File: schematic/incremental-buzzer.sch (KiCad schematic (older format))
At the start: 50 parts, among them Q1 PNP, U1 4051, U2 4013, U3 4040, U4 4584, U5 4013

Commit message: changed pull-down resistor
Parts:
- R18: value 100K -> 10K
Changed lines of the file:
@@
 Sheet 1 1
 Title "INCREMENTAL VOLUME ALARM WITH SNOOZE"
-Date "2 mar 2016"
-Rev "5"
+Date "18 apr 2016"
+Rev "6"
 Comp "Michael Craft"
 Comment1 ""
@@
 P 1850 5450
 F 0 "R18" V 1930 5450 40  0000 C CNN
-F 1 "100K" V 1750 5450 40  0000 C CNN
+F 1 "10K" V 1750 5450 40  0000 C CNN
 F 2 "~" V 1780 5450 30  0000 C CNN
 F 3 "~" H 1850 5450 30  0000 C CNN

Commit message: enhanced input protection
Parts:
- added C?: 1uF, ~, symbol C
- added R?: 1K, ~, symbol USR
Connections:
- net +5V: now also C?.2, R?.1, R?.2
- net GND: now also C?.1
Changed lines of the file:
@@
 Title "INCREMENTAL VOLUME ALARM WITH SNOOZE"
 Date "18 apr 2016"
-Rev "6"
+Rev "7"
 Comp "Michael Craft"
 Comment1 ""
@@
 L +5V #PWR22
 U 1 1 56CCB88D
-P 1850 4950
-F 0 "#PWR22" H 1850 5040 20  0001 C CNN
-F 1 "+5V" H 1850 5040 30  0000 C CNN
-F 2 "" H 1850 4950 60  0000 C CNN
-F 3 "" H 1850 4950 60  0000 C CNN
-	1    1850 4950
+P 1800 4500
+F 0 "#PWR22" H 1800 4590 20  0001 C CNN
+F 1 "+5V" H 1800 4590 30  0000 C CNN
+F 2 "" H 1800 4500 60  0000 C CNN
+F 3 "" H 1800 4500 60  0000 C CNN
+	1    1800 4500
 	1    0    0    -1
 $EndComp
@@
 L USGND #PWR27
 U 1 1 56CCC9B7
-P 1850 5750
-F 0 "#PWR27" H 1850 5750 30  0001 C CNN
-F 1 "GND" H 1850 5680 30  0001 C CNN
-F 2 "" H 1850 5750 60  0000 C CNN
-F 3 "" H 1850 5750 60  0000 C CNN
-	1    1850 5750
+P 1850 6000
+F 0 "#PWR27" H 1850 6000 30  0001 C CNN
+F 1 "GND" H 1850 5930 30  0001 C CNN
+F 2 "" H 1850 6000 60  0000 C CNN
+F 3 "" H 1850 6000 60  0000 C CNN
+	1    1850 6000
 	1    0    0    -1
 $EndComp
@@
 	1900 1400 1900 1350
 Wire Wire Line
-	1700 5000 1850 5000
-Wire Wire Line
-	1850 5000 1850 4950
-Wire Wire Line
 	5800 3150 5800 3300
 Wire Wire Line
@@
 	6400 6500 700  6500
 Wire Wire Line
-	1850 5700 1850 5750
+	1850 5700 1850 6000
 Wire Wire Line
 	2350 7050 2400 7050
@@
 Connection ~ 4750 2450
 Connection ~ 2900 2500
-Connection ~ 1850 5750
+Connection ~ 1850 6000
 Connection ~ 1400 7450
 Connection ~ 2350 7250
@@
 Wire Wire Line
 	9750 2350 9700 2350
+$Comp
+L C C?
+U 1 1 5714C6E0
+P 1650 5800
+F 0 "C?" H 1650 5900 40  0000 L CNN
+F 1 "1uF" H 1656 5715 40  0000 L CNN
+F 2 "~" H 1688 5650 30  0000 C CNN
+F 3 "~" H 1650 5800 60  0000 C CNN
+	1    1650 5800
+	0    1    1    0
+$EndComp
+Connection ~ 1850 5800
+$Comp
+L +5V #PWR?
+U 1 1 5714C700
+P 1400 5750
+F 0 "#PWR?" H 1400 5840 20  0001 C CNN
+F 1 "+5V" H 1400 5840 30  0000 C CNN
+F 2 "" H 1400 5750 60  0000 C CNN
+F 3 "" H 1400 5750 60  0000 C CNN
+	1    1400 5750
+	1    0    0    -1
+$EndComp
+Wire Wire Line
+	1400 5750 1400 5800
+Wire Wire Line
+	1400 5800 1450 5800
+$Comp
+L USR R?
+U 1 1 5714C9DD
+P 1800 4750
+F 0 "R?" V 1880 4750 40  0000 C CNN
+F 1 "1K" V 1700 4750 40  0000 C CNN
+F 2 "~" V 1730 4750 30  0000 C CNN
+F 3 "~" H 1800 4750 30  0000 C CNN
+	1    1800 4750
+	-1   0    0    1
+$EndComp
+Wire Wire Line
+	1700 5000 1800 5000
+Connection ~ 1800 4500
 $EndSCHEMATC

Commit message: better volume ramp
Parts:
- R1: value 27K -> 470K
- R2: value 27K -> 330K
- R3: value 27K -> 180K
- R4: value 18K -> 100K
- R5: value 18K -> 56K
- R6: value 18K -> 33K
- R8: value 18K -> 10K
- gave numbers to parts that had none: 2
- renumbered C6 to C7, C7 to C8, R16 to R17, R17 to R18, R18 to R19, R19 to R20, R20 to R21
Connections:
- net GND: now also R1.2, R2.2, R3.2, R4.2, R5.2, R6.2, R7.2, R8.2; no longer R8.1
- net at U1.13 (X0): now also R1.1; no longer R1.2
- new net: R5.1, U1.1 (X4)
- new net: R4.1, U1.12 (X3)
- new net: R2.1, U1.14 (X1)
- new net: R3.1, U1.15 (X2)
- new net: R7.1, U1.2 (X6)
- new net: R8.1, U1.4 (X7)
- new net: R6.1, U1.5 (X5)
Other:
- moved on the sheet: R8
