File: schematic/incremental-buzzer.sch (KiCad schematic (older format))
At the start: 52 parts, among them Q1 PNP, U1 4051, U2 4013, U3 4040, U4 4584, U5 4013

Commit message: schematic is "done"
Parts:
- removed R16: 1K, ~, symbol USR
