File: schematic/incremental-buzzer.sch (KiCad schematic (older format))
At the start: 51 parts, among them Q1 PNP, U1 4051, U2 4013, U3 4040, U4 4584, U5 4013

Commit message: passes ERC
Parts:
- renumbered R17 to R16, R18 to R17, R19 to R18, R20 to R19, R21 to R20
