File: schematic/display-board.sch (KiCad schematic (older format))
At the start: 2 parts

Commit message: cleanup kicad project
Parts:
- added P1: 4-PIN_HEADER, ~, symbol 4-PIN_HEADER
- gave numbers to parts that had none: 2
Connections:
- net labels added: +5V, GND, VCC
- wire segments 0 -> 7
Changed lines of the file:
@@
 Sheet 1 1
 Title ""
-Date "23 mar 2016"
+Date "30 may 2016"
 Rev ""
 Comp ""
@@
 $EndDescr
 $Comp
-L 7SEG-KB AFF?
+L 7SEG-KB AFF1
 U 1 1 56F2F8F8
 P 10300 1400
-F 0 "AFF?" H 10300 1950 60  0000 C CNN
-F 1 "7SEG-KB" H 10300 950 60  0000 C CNN
+F 0 "AFF1" H 10300 1950 60  0000 C CNN
+F 1 "7SEG-KB" H 10300 700 60  0000 C CNN
 F 2 "~" H 10300 1500 60  0000 C CNN
 F 3 "~" H 10300 1500 60  0000 C CNN
@@
 $EndComp
 $Comp
-L 4511 U?
+L 4511 U1
 U 1 1 56F30351
 P 9000 1500
-F 0 "U?" H 9350 2150 60  0000 C CNN
+F 0 "U1" H 9350 2150 60  0000 C CNN
 F 1 "4511" H 9200 850 60  0000 C CNN
 F 2 "~" H 9000 1500 60  0000 C CNN
@@
 	1    0    0    -1
 $EndComp
-Connection ~ 9700 1000
-Connection ~ 9700 1100
-Connection ~ 9700 1200
-Connection ~ 9700 1300
-Connection ~ 9700 1400
-Connection ~ 9700 1500
-Connection ~ 9700 1600
 NoConn ~ 10900 1550
 $Comp
-L USGND #PWR?
+L USGND #PWR01
 U 1 1 56F3037A
 P 10900 1750
-F 0 "#PWR?" H 10900 1750 30  0001 C CNN
+F 0 "#PWR01" H 10900 1750 30  0001 C CNN
 F 1 "USGND" H 10900 1680 30  0001 C CNN
 F 2 "~" H 10900 1750 60  0000 C CNN
@@
 	0    -1   -1   0
 $EndComp
+Connection ~ 9700 1000
+Connection ~ 9700 1100
+Connection ~ 9700 1200
+Connection ~ 9700 1300
+Connection ~ 9700 1400
+Connection ~ 9700 1600
 Connection ~ 10900 1750
+$Comp
+L +5V #PWR02
+U 1 1 57333E03
+P 6800 1450
+F 0 "#PWR02" H 6800 1540 20  0001 C CNN
+F 1 "+5V" H 6800 1540 30  0000 C CNN
+F 2 "" H 6800 1450 60  0000 C CNN
+F 3 "" H 6800 1450 60  0000 C CNN
+	1    6800 1450
+	1    0    0    -1
+$EndComp
+$Comp
+L USGND #PWR03
+U 1 1 57333E23
+P 8300 1800
+F 0 "#PWR03" H 8300 1800 30  0001 C CNN
+F 1 "USGND" H 8300 1730 30  0001 C CNN
+F 2 "~" H 8300 1800 60  0000 C CNN
+F 3 "~" H 8300 1800 60  0000 C CNN
+	1    8300 1800
+	1    0    0    -1
+$EndComp
+Wire Wire Line
+	8300 1650 8300 1800
+Wire Wire Line
+	8300 1450 6800 1450
+Wire Wire Line
+	8300 1450 8300 1550
+$Comp
+L PWR_FLAG #FLG04
+U 1 1 573340A9
+P 8150 1900
+F 0 "#FLG04" H 8150 1995 30  0001 C CNN
+F 1 "PWR_FLAG" H 8150 2080 30  0000 C CNN
+F 2 "" H 8150 1900 60  0000 C CNN
+F 3 "" H 8150 1900 60  0000 C CNN
+	1    8150 1900
+	-1   0    0    1
+$EndComp
+Wire Wire Line
+	8150 1900 8150 1750
+Wire Wire Line
+	8100 1750 8300 1750
+Connection ~ 8300 1750
+$Comp
+L PWR_FLAG #FLG05
+U 1 1 573340CE
+P 6950 1350
+F 0 "#FLG05" H 6950 1445 30  0001 C CNN
+F 1 "PWR_FLAG" H 6950 1530 30  0000 C CNN
+F 2 "" H 6950 1350 60  0000 C CNN
+F 3 "" H 6950 1350 60  0000 C CNN
+	1    6950 1350
+	1    0    0    -1
+$EndComp
+Wire Wire Line
+	6950 1350 6950 1650
+Connection ~ 6950 1450
+Connection ~ 9700 1500
+$Comp
+L VCC #PWR06
+U 1 1 57334183
+P 6950 1650
+F 0 "#PWR06" H 6950 1750 30  0001 C CNN
+F 1 "VCC" H 6950 1750 30  0000 C CNN
+F 2 "" H 6950 1650 60  0000 C CNN
+F 3 "" H 6950 1650 60  0000 C CNN
+	1    6950 1650
+	-1   0    0    1
+$EndComp
+$Comp
+L 4-PIN_HEADER P1
+U 1 1 574BA340
+P 8050 1150
+F 0 "P1" H 7700 1150 50  0000 C CNN
+F 1 "4-PIN_HEADER" H 8100 1350 50  0001 C CNN
+F 2 "~" H 8150 1300 60  0000 C CNN
+F 3 "~" H 8150 1300 60  0000 C CNN
+	1    8050 1150
+	0    -1   1    0
+$EndComp
+Connection ~ 8300 1000
+Connection ~ 8300 1100
+Connection ~ 8300 1200
+Connection ~ 8300 1300
+Connection ~ 8300 1450
+Wire Wire Line
+	10900 1750 10900 1950
+Connection ~ 10900 1850
+$Comp
+L GND #PWR07
+U 1 1 574BAA45
+P 8100 1750
+F 0 "#PWR07" H 8100 1750 30  0001 C CNN
+F 1 "GND" H 8100 1680 30  0001 C CNN
+F 2 "" H 8100 1750 60  0000 C CNN
+F 3 "" H 8100 1750 60  0000 C CNN
+	1    8100 1750
+	0    1    1    0
+$EndComp
+Connection ~ 8150 1750
 $EndSCHEMATC

Commit message: cleaned up kicad project more
Parts:
- added P3: 2-PIN_HEADER, ~, symbol 2-PIN_HEADER
- renumbered P1 to P2, U1 to U6
Connections:
- net labels added: 0A, 0B, 0C, 0D
- net labels removed: VCC
- wire segments 7 -> 17
Changed lines of the file:
@@
 LIBS:valves
 LIBS:kicad-custom-parts
+LIBS:logic-clock-cache
 EELAYER 27 0
 EELAYER END
 $Descr A4 11693 8268
 encoding utf-8
-Sheet 1 1
+Sheet 3 4
 Title ""
 Date "30 may 2016"
@@
 Comment4 ""
 $EndDescr
+$Comp
+L 4511 U6
+U 1 1 56F30351
+P 9000 1500
+F 0 "U6" H 9350 2150 60  0000 C CNN
+F 1 "4511" H 9200 850 60  0000 C CNN
+F 2 "~" H 9000 1500 60  0000 C CNN
+F 3 "~" H 9000 1500 60  0000 C CNN
+	1    9000 1500
+	1    0    0    -1
+$EndComp
+NoConn ~ 10900 1550
+$Comp
+L USGND #PWR057
+U 1 1 56F3037A
+P 10900 1750
+F 0 "#PWR057" H 10900 1750 30  0001 C CNN
+F 1 "USGND" H 10900 1680 30  0001 C CNN
+F 2 "~" H 10900 1750 60  0000 C CNN
+F 3 "~" H 10900 1750 60  0000 C CNN
+	1    10900 1750
+	0    -1   -1   0
+$EndComp
+$Comp
+L USGND #PWR058
+U 1 1 57333E23
+P 8300 1800
+F 0 "#PWR058" H 8300 1800 30  0001 C CNN
+F 1 "USGND" H 8300 1730 30  0001 C CNN
+F 2 "~" H 8300 1800 60  0000 C CNN
+F 3 "~" H 8300 1800 60  0000 C CNN
+	1    8300 1800
+	1    0    0    -1
+$EndComp
+$Comp
+L 4-PIN_HEADER P2
+U 1 1 574BA340
+P 6200 1700
+F 0 "P2" H 5850 1700 50  0000 C CNN
+F 1 "4-PIN_HEADER" H 6250 1900 50  0001 C CNN
+F 2 "~" H 6300 1850 60  0000 C CNN
+F 3 "~" H 6300 1850 60  0000 C CNN
+	1    6200 1700
+	1    0    0    1
+$EndComp
+Text HLabel 6050 1800 3    60   Input ~ 0
+0A
+Text HLabel 6150 1800 3    60   Input ~ 0
+0B
+Text HLabel 6250 1800 3    60   Input ~ 0
+0C
+Text HLabel 6350 1800 3    60   Input ~ 0
+0D
 $Comp
 L 7SEG-KB AFF1
@@
 	1    0    0    -1
 $EndComp
-$Comp
-L 4511 U1
-U 1 1 56F30351
-P 9000 1500
-F 0 "U1" H 9350 2150 60  0000 C CNN
-F 1 "4511" H 9200 850 60  0000 C CNN
-F 2 "~" H 9000 1500 60  0000 C CNN
-F 3 "~" H 9000 1500 60  0000 C CNN
-	1    9000 1500
-	1    0    0    -1
-$EndComp
-NoConn ~ 10900 1550
-$Comp
-L USGND #PWR01
-U 1 1 56F3037A
-P 10900 1750
-F 0 "#PWR01" H 10900 1750 30  0001 C CNN
-F 1 "USGND" H 10900 1680 30  0001 C CNN
-F 2 "~" H 10900 1750 60  0000 C CNN
-F 3 "~" H 10900 1750 60  0000 C CNN
-	1    10900 1750
-	0    -1   -1   0
-$EndComp
 Connection ~ 9700 1000
 Connection ~ 9700 1100
@@
 Connection ~ 9700 1600
 Connection ~ 10900 1750
-$Comp
-L +5V #PWR02
-U 1 1 57333E03
-P 6800 1450
-F 0 "#PWR02" H 6800 1540 20  0001 C CNN
-F 1 "+5V" H 6800 1540 30  0000 C CNN
-F 2 "" H 6800 1450 60  0000 C CNN
-F 3 "" H 6800 1450 60  0000 C CNN
-	1    6800 1450
-	1    0    0    -1
-$EndComp
-$Comp
-L USGND #PWR03
-U 1 1 57333E23
-P 8300 1800
-F 0 "#PWR03" H 8300 1800 30  0001 C CNN
-F 1 "USGND" H 8300 1730 30  0001 C CNN
-F 2 "~" H 8300 1800 60  0000 C CNN
-F 3 "~" H 8300 1800 60  0000 C CNN
-	1    8300 1800
-	1    0    0    -1
-$EndComp
 Wire Wire Line
 	8300 1650 8300 1800
 Wire Wire Line
-	8300 1450 6800 1450
-Wire Wire Line
 	8300 1450 8300 1550
-$Comp
-L PWR_FLAG #FLG04
-U 1 1 573340A9
-P 8150 1900
-F 0 "#FLG04" H 8150 1995 30  0001 C CNN
-F 1 "PWR_FLAG" H 8150 2080 30  0000 C CNN
-F 2 "" H 8150 1900 60  0000 C CNN
-F 3 "" H 8150 1900 60  0000 C CNN
-	1    8150 1900
-	-1   0    0    1
-$EndComp
-Wire Wire Line
-	8150 1900 8150 1750
-Wire Wire Line
-	8100 1750 8300 1750
 Connection ~ 8300 1750
-$Comp
-L PWR_FLAG #FLG05
-U 1 1 573340CE
-P 6950 1350
-F 0 "#FLG05" H 6950 1445 30  0001 C CNN
-F 1 "PWR_FLAG" H 6950 1530 30  0000 C CNN
-F 2 "" H 6950 1350 60  0000 C CNN
-F 3 "" H 6950 1350 60  0000 C CNN
-	1    6950 1350
-	1    0    0    -1
-$EndComp
-Wire Wire Line
-	6950 1350 6950 1650
-Connection ~ 6950 1450
 Connection ~ 9700 1500
-$Comp
-L VCC #PWR06
-U 1 1 57334183
-P 6950 1650
-F 0 "#PWR06" H 6950 1750 30  0001 C CNN
-F 1 "VCC" H 6950 1750 30  0000 C CNN
-F 2 "" H 6950 1650 60  0000 C CNN
-F 3 "" H 6950 1650 60  0000 C CNN
-	1    6950 1650
-	-1   0    0    1
-$EndComp
-$Comp
-L 4-PIN_HEADER P1
-U 1 1 574BA340
-P 8050 1150
-F 0 "P1" H 7700 1150 50  0000 C CNN
-F 1 "4-PIN_HEADER" H 8100 1350 50  0001 C CNN
-F 2 "~" H 8150 1300 60  0000 C CNN
-F 3 "~" H 8150 1300 60  0000 C CNN
-	1    8050 1150
-	0    -1   1    0
-$EndComp
-Connection ~ 8300 1000
-Connection ~ 8300 1100
-Connection ~ 8300 1200
-Connection ~ 8300 1300
 Connection ~ 8300 1450
 Wire Wire Line
@@
 Connection ~ 10900 1850
 $Comp
-L GND #PWR07
-U 1 1 574BAA45
-P 8100 1750
-F 0 "#PWR07" H 8100 1750 30  0001 C CNN
-F 1 "GND" H 8100 1680 30  0001 C CNN
-F 2 "" H 8100 1750 60  0000 C CNN
-F 3 "" H 8100 1750 60  0000 C CNN
-	1    8100 1750
-	0    1    1    0
+L 2-PIN_HEADER P3
+U 1 1 574BC3AE
+P 7450 1800
+F 0 "P3" H 7200 1800 50  0000 C CNN
+F 1 "2-PIN_HEADER" H 7450 1900 50  0001 C CNN
+F 2 "~" H 7550 1950 60  0000 C CNN
+F 3 "~" H 7550 1950 60  0000 C CNN
+	1    7450 1800
+	0    -1   1    0
 $EndComp
-Connection ~ 8150 1750
+Wire Wire Line
+	7700 1750 7700 1450
+Wire Wire Line
+	7350 1850 8150 1850
+Text HLabel 7350 1750 0    60   Input ~ 0
++5V
+Text HLabel 7350 1850 0    60   UnSpc ~ 0
+GND
+Wire Wire Line
+	7700 1750 7350 1750
+Connection ~ 7700 1850
+Wire Wire Line
+	8300 1000 6050 1000
+Wire Wire Line
+	6050 1000 6050 1800
+Wire Wire Line
+	8300 1100 6150 1100
+Wire Wire Line
+	6150 1100 6150 1800
+Wire Wire Line
+	8300 1200 6250 1200
+Wire Wire Line
+	6250 1200 6250 1800
+Wire Wire Line
+	8300 1300 6350 1300
+Wire Wire Line
+	6350 1300 6350 1800
+Connection ~ 6050 1450
+Connection ~ 6150 1450
+Connection ~ 6250 1450
+Connection ~ 6350 1450
+Wire Wire Line
+	8300 1750 8150 1750
+Wire Wire Line
+	8150 1750 8150 1850
+Wire Wire Line
+	7700 1450 8300 1450
 $EndSCHEMATC

Commit message: started pcb
Parts:
- renumbered P2 to P5, P3 to P6
Connections:
- wire segments 17 -> 16
Changed lines of the file:
@@
 LIBS:valves
 LIBS:kicad-custom-parts
-LIBS:logic-clock-cache
 EELAYER 27 0
 EELAYER END
@@
 NoConn ~ 10900 1550
 $Comp
-L USGND #PWR057
+L USGND #PWR058
 U 1 1 56F3037A
 P 10900 1750
-F 0 "#PWR057" H 10900 1750 30  0001 C CNN
+F 0 "#PWR058" H 10900 1750 30  0001 C CNN
 F 1 "USGND" H 10900 1680 30  0001 C CNN
 F 2 "~" H 10900 1750 60  0000 C CNN
@@
 $EndComp
 $Comp
-L USGND #PWR058
-U 1 1 57333E23
-P 8300 1800
-F 0 "#PWR058" H 8300 1800 30  0001 C CNN
-F 1 "USGND" H 8300 1730 30  0001 C CNN
-F 2 "~" H 8300 1800 60  0000 C CNN
-F 3 "~" H 8300 1800 60  0000 C CNN
-	1    8300 1800
-	1    0    0    -1
-$EndComp
-$Comp
-L 4-PIN_HEADER P2
+L 4-PIN_HEADER P5
 U 1 1 574BA340
 P 6200 1700
-F 0 "P2" H 5850 1700 50  0000 C CNN
+F 0 "P5" H 5850 1700 50  0000 C CNN
 F 1 "4-PIN_HEADER" H 6250 1900 50  0001 C CNN
 F 2 "~" H 6300 1850 60  0000 C CNN
@@
 Connection ~ 10900 1750
 Wire Wire Line
-	8300 1650 8300 1800
-Wire Wire Line
 	8300 1450 8300 1550
-Connection ~ 8300 1750
 Connection ~ 9700 1500
 Connection ~ 8300 1450
@@
 Connection ~ 10900 1850
 $Comp
-L 2-PIN_HEADER P3
+L 2-PIN_HEADER P6
 U 1 1 574BC3AE
 P 7450 1800
-F 0 "P3" H 7200 1800 50  0000 C CNN
+F 0 "P6" H 7200 1800 50  0000 C CNN
 F 1 "2-PIN_HEADER" H 7450 1900 50  0001 C CNN
 F 2 "~" H 7550 1950 60  0000 C CNN
@@
 	7700 1750 7700 1450
 Wire Wire Line
-	7350 1850 8150 1850
+	7350 1850 8300 1850
 Text HLabel 7350 1750 0    60   Input ~ 0
 +5V
@@
 Connection ~ 6350 1450
 Wire Wire Line
-	8300 1750 8150 1750
+	7300 1450 8300 1450
 Wire Wire Line
-	8150 1750 8150 1850
+	8300 1850 8300 1650
+Text GLabel 7900 1950 3    60   UnSpc ~ 0
+GND
 Wire Wire Line
-	7700 1450 8300 1450
+	7900 1950 7900 1850
+Connection ~ 7900 1850
+Text GLabel 7300 1450 0    60   UnSpc ~ 0
++5V
+Connection ~ 7700 1450
 $EndSCHEMATC

Commit message: display board schematic
Parts:
- added AFF?: SECONDS, ~, symbol 7SEG-KB
- added AFF?: TEN-SECONDS, ~, symbol 7SEG-KB
- added AFF?: MINUTES, ~, symbol 7SEG-KB
- added AFF?: TEN-MINUTES, ~, symbol 7SEG-KB
- added AFF?: HOURS, ~, symbol 7SEG-KB
- added AFF?: TEN-HOURS, ~, symbol 7SEG-KB
- added AFF?: AM-PM, ~, symbol 7SEG-KB
- added D? (x4): LED, ~, symbol LED
- added P? (x5): 4-PIN_HEADER, ~, symbol 4-PIN_HEADER
- added P?: 2-PIN_HEADER, ~, symbol 2-PIN_HEADER
- added Q?: ZVN4206, ~, symbol MOS_N
- added Q?: MOS_P, ~, symbol MOS_P
- added R? (x5): 1K, ~, symbol USR
- added U? (x5): 4511, ~, symbol 4511
- AFF1: value 7SEG-KB -> TENTH-SECONDS
Connections:
- net labels added: 1A, 1B, 1C, 1D, 2A, 2B, 2C, 2D, 3A, 3B, 3C, 3D, 4A, 4B, 4C, 4D, 5A, 5B, 5C, 5D, AM, TEN-HR
- wire segments 16 -> 96
- no-connect marks 1 -> 13
Other:
- note added: "HOURS"
- note added: "MINUTES"
- note added: "SECONDS"
- moved on the sheet: AFF1, U6

Commit message: pcb rev 1
Parts:
- added C12, C13, C14, C15, C16, C17: 100nF BYPASS, ~, symbol CSMALL
- gave numbers to parts that had none: 29
Connections:
- wire segments 96 -> 119
Other:
- moved on the sheet: U13

Commit message: lots of stuff
Parts:
- R27: value 1K -> 56R
- R28: value 1K -> 27R
- R29, R30, R31: value 1K -> 470R
Changed lines of the file:
@@
 Sheet 4 4
 Title "LOGIC CLOCK DISPLAY BOARD"
-Date "30 may 2016"
-Rev "1"
+Date "20 jun 2016"
+Rev "3"
 Comp "Michael Craft"
 Comment1 ""
@@
 P 10300 4900
 F 0 "R30" V 10380 4900 40  0000 C CNN
-F 1 "1K" V 10200 4900 40  0000 C CNN
+F 1 "470R" V 10200 4900 40  0000 C CNN
 F 2 "~" V 10230 4900 30  0000 C CNN
 F 3 "~" H 10300 4900 30  0000 C CNN
@@
 P 7150 6200
 F 0 "R31" V 7230 6200 40  0000 C CNN
-F 1 "1K" V 7050 6200 40  0000 C CNN
+F 1 "470R" V 7050 6200 40  0000 C CNN
 F 2 "~" V 7080 6200 30  0000 C CNN
 F 3 "~" H 7150 6200 30  0000 C CNN
@@
 P 10300 3450
 F 0 "R29" V 10380 3450 40  0000 C CNN
-F 1 "1K" V 10200 3450 40  0000 C CNN
+F 1 "470R" V 10200 3450 40  0000 C CNN
 F 2 "~" V 10230 3450 30  0000 C CNN
 F 3 "~" H 10300 3450 30  0000 C CNN
@@
 P 6750 3200
 F 0 "R28" V 6830 3200 40  0000 C CNN
-F 1 "1K" V 6650 3200 40  0000 C CNN
+F 1 "27R" V 6650 3200 40  0000 C CNN
 F 2 "~" V 6680 3200 30  0000 C CNN
 F 3 "~" H 6750 3200 30  0000 C CNN
@@
 P 4950 3200
 F 0 "R27" V 5030 3200 40  0000 C CNN
-F 1 "1K" V 4850 3200 40  0000 C CNN
+F 1 "56R" V 4850 3200 40  0000 C CNN
 F 2 "~" V 4880 3200 30  0000 C CNN
 F 3 "~" H 4950 3200 30  0000 C CNN

Commit message: working on schematic...
Connections:
- net labels added: DISPLAY_PWM_SINK, DPS
- net labels removed: GND, USGND
- wire segments 119 -> 137
