File: schematic/display-board.sch (KiCad schematic (older format))
At the start: 39 parts, among them P13 2-PIN_HEADER, P14 4-PIN_HEADER, P15 4-PIN_HEADER, P16 4-PIN_HEADER, P17 4-PIN_HEADER, P18 4-PIN_HEADER, P5 4-PIN_HEADER, P6 2-PIN_HEADER, Q2 MOS_P, Q3 ZVN4206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

Commit message: passes ERC
Parts:
- renumbered AFF2 to AFF1, AFF3 to AFF2, AFF4 to AFF3, AFF5 to AFF4, AFF6 to AFF5, AFF7 to AFF6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
