File: schematic/power-board.sch (KiCad schematic (older format))
At the start: 16 parts

Commit message: cleaned up kicad project more
Parts:
- added R24: 0, ~, symbol USR
- gave numbers to parts that had none: 16
Connections:
- net labels added: USGND
- wire segments 32 -> 34
Changed lines of the file:
@@
 LIBS:valves
 LIBS:kicad-custom-parts
-LIBS:power-board-cache
+LIBS:logic-clock-cache
 EELAYER 27 0
 EELAYER END
 $Descr USLetter 11000 8500
 encoding utf-8
-Sheet 1 1
+Sheet 4 4
 Title "60Hz LOW VOLTAGE AC TO DC SUPPLY W/ 10Hz OUT"
-Date "23 feb 2016"
+Date "30 may 2016"
 Rev "2"
 Comp ""
@@
 Connection ~ 4300 3950
 Wire Wire Line
-	4800 3650 4800 4650
-$Comp
-L GND #PWR?
-U 1 1 56AE936F
-P 4800 4650
-F 0 "#PWR?" H 4800 4650 30  0001 C CNN
-F 1 "GND" H 4800 4580 30  0001 C CNN
-F 2 "" H 4800 4650 60  0000 C CNN
-F 3 "" H 4800 4650 60  0000 C CNN
-	1    4800 4650
-	1    0    0    -1
-$EndComp
+	4800 5200 4800 3650
 Connection ~ 4800 3950
 Wire Wire Line
 	3700 3650 3700 4300
 $Comp
-L CP1 C?
+L CP1 C9
 U 1 1 56AE939E
 P 4300 4300
-F 0 "C?" H 4350 4400 50  0000 L CNN
+F 0 "C9" H 4350 4400 50  0000 L CNN
 F 1 "220uF" H 4350 4200 50  0000 L CNN
 F 2 "~" H 4300 4300 60  0000 C CNN
@@
 Connection ~ 3700 3950
 $Comp
-L 7805 U?
+L 7805 U8
 U 1 1 56AE9417
 P 3300 4350
-F 0 "U?" H 3450 4154 60  0000 C CNN
+F 0 "U8" H 3450 4154 60  0000 C CNN
 F 1 "7805" H 3300 4550 60  0000 C CNN
 F 2 "" H 3300 4350 60  0000 C CNN
@@
 $EndComp
 Connection ~ 3700 4300
-$Comp
-L GND #PWR?
-U 1 1 56AE942E
-P 3300 4650
-F 0 "#PWR?" H 3300 4650 30  0001 C CNN
-F 1 "GND" H 3300 4580 30  0001 C CNN
-F 2 "" H 3300 4650 60  0000 C CNN
-F 3 "" H 3300 4650 60  0000 C CNN
-	1    3300 4650
-	1    0    0    -1
-$EndComp
-Wire Wire Line
-	3300 4600 3300 4650
-$Comp
-L GND #PWR?
-U 1 1 56AE9482
-P 2900 4650
-F 0 "#PWR?" H 2900 4650 30  0001 C CNN
-F 1 "GND" H 2900 4580 30  0001 C CNN
-F 2 "" H 2900 4650 60  0000 C CNN
-F 3 "" H 2900 4650 60  0000 C CNN
-	1    2900 4650
-	1    0    0    -1
-$EndComp
-$Comp
-L CSMALL C?
+Wire Wire Line
+	3300 4600 3300 5200
+$Comp
+L CSMALL C10
 U 1 1 56AE9499
 P 2900 4450
-F 0 "C?" H 2925 4500 30  0000 L CNN
+F 0 "C10" H 2925 4500 30  0000 L CNN
 F 1 "1uF" H 2925 4400 30  0000 L CNN
 F 2 "~" H 2900 4450 60  0000 C CNN
@@
 $EndComp
 Wire Wire Line
-	2900 3300 2900 4350
-Wire Wire Line
-	2900 4550 2900 4650
-$Comp
-L +5V #PWR?
+	2900 4550 2900 5200
+$Comp
+L +5V #PWR059
 U 1 1 56AE94DA
-P 2900 3300
-F 0 "#PWR?" H 2900 3390 20  0001 C CNN
-F 1 "+5V" H 2900 3390 30  0000 C CNN
-F 2 "" H 2900 3300 60  0000 C CNN
-F 3 "" H 2900 3300 60  0000 C CNN
-	1    2900 3300
-	1    0    0    -1
-$EndComp
-Connection ~ 2900 4300
+P 2900 3400
+F 0 "#PWR059" H 2900 3490 20  0001 C CNN
+F 1 "+5V" H 2900 3490 30  0000 C CNN
+F 2 "" H 2900 3400 60  0000 C CNN
+F 3 "" H 2900 3400 60  0000 C CNN
+	1    2900 3400
+	1    0    0    -1
+$EndComp
 Wire Notes Line
 	4100 3000 4100 3350
@@
 	4400 3000 4100 3000
 $Comp
-L 4040 U?
+L 4040 U7
 U 1 1 56AE9575
 P 6350 3950
-F 0 "U?" H 6450 4600 60  0000 C CNN
+F 0 "U7" H 6450 4600 60  0000 C CNN
 F 1 "4040" H 6600 3300 60  0000 C CNN
 F 2 "" H 6350 3950 60  0000 C CNN
@@
 Connection ~ 4300 3400
 $Comp
-L USR R?
+L USR R23
 U 1 1 56AE976F
 P 5050 3400
-F 0 "R?" V 5130 3400 40  0000 C CNN
+F 0 "R23" V 5130 3400 40  0000 C CNN
 F 1 "2K7" V 4950 3400 40  0000 C CNN
 F 2 "~" V 4980 3400 30  0000 C CNN
@@
 Connection ~ 4800 3400
 $Comp
-L USR R?
+L USR R25
 U 1 1 56AE9781
 P 5300 3950
-F 0 "R?" V 5380 3950 40  0000 C CNN
+F 0 "R25" V 5380 3950 40  0000 C CNN
 F 1 "1K" V 5200 3950 40  0000 C CNN
 F 2 "~" V 5230 3950 30  0000 C CNN
@@
 Wire Wire Line
 	5300 3400 5300 3700
-$Comp
-L GND #PWR?
-U 1 1 56AE97A8
-P 5300 4650
-F 0 "#PWR?" H 5300 4650 30  0001 C CNN
-F 1 "GND" H 5300 4580 30  0001 C CNN
-F 2 "" H 5300 4650 60  0000 C CNN
-F 3 "" H 5300 4650 60  0000 C CNN
-	1    5300 4650
-	1    0    0    -1
-$EndComp
-Wire Wire Line
-	5300 4200 5300 4650
+Wire Wire Line
+	5300 4200 5300 5250
 Wire Wire Line
 	5300 3400 5700 3400
 $Comp
-L CSMALL C?
+L CSMALL C11
 U 1 1 56AE9894
 P 6300 5050
-F 0 "C?" H 6325 5100 30  0000 L CNN
+F 0 "C11" H 6325 5100 30  0000 L CNN
 F 1 "100nF BYPASS" H 6325 5000 30  0000 L CNN
 F 2 "~" H 6300 5050 60  0000 C CNN
@@
 $EndComp
 $Comp
-L +5V #PWR?
+L +5V #PWR060
 U 1 1 56AE98AF
 P 6300 4900
-F 0 "#PWR?" H 6300 4990 20  0001 C CNN
+F 0 "#PWR060" H 6300 4990 20  0001 C CNN
 F 1 "+5V" H 6300 4990 30  0000 C CNN
 F 2 "" H 6300 4900 60  0000 C CNN
@@
 Wire Wire Line
 	6300 4950 6300 4900
-$Comp
-L GND #PWR?
-U 1 1 56AE98E5
-P 6300 5200
-F 0 "#PWR?" H 6300 5200 30  0001 C CNN
-F 1 "GND" H 6300 5130 30  0001 C CNN
-F 2 "" H 6300 5200 60  0000 C CNN
-F 3 "" H 6300 5200 60  0000 C CNN
-	1    6300 5200
-	1    0    0    -1
-$EndComp
-Wire Wire Line
-	6300 5150 6300 5200
+Wire Wire Line
+	6300 5200 6300 5150
 NoConn ~ 7000 3400
 NoConn ~ 7000 3500
@@
 NoConn ~ 7000 4500
 $Comp
-L DIODE D?
+L DIODE D17
 U 1 1 56AE9A06
 P 7350 3600
-F 0 "D?" H 7350 3700 40  0000 C CNN
+F 0 "D17" H 7350 3700 40  0000 C CNN
 F 1 "DIODE" H 7350 3500 40  0001 C CNN
 F 2 "~" H 7350 3600 60  0000 C CNN
@@
 $EndComp
 $Comp
-L DIODE D?
+L DIODE D20
 U 1 1 56AE9A11
 P 7350 3750
-F 0 "D?" H 7350 3850 40  0000 C CNN
+F 0 "D20" H 7350 3850 40  0000 C CNN
 F 1 "DIODE" H 7350 3650 40  0001 C CNN
 F 2 "~" H 7350 3750 60  0000 C CNN
@@
 Connection ~ 7550 3750
 $Comp
-L USR R?
+L USR R22
 U 1 1 56AE9AD5
 P 7550 3300
-F 0 "R?" V 7630 3300 40  0000 C CNN
+F 0 "R22" V 7630 3300 40  0000 C CNN
 F 1 "100K" V 7450 3300 40  0000 C CNN
 F 2 "~" V 7480 3300 30  0000 C CNN
@@
 $EndComp
 $Comp
-L +5V #PWR?
+L +5V #PWR061
 U 1 1 56AE9ADB
 P 7550 3000
-F 0 "#PWR?" H 7550 3090 20  0001 C CNN
+F 0 "#PWR061" H 7550 3090 20  0001 C CNN
 F 1 "+5V" H 7550 3090 30  0000 C CNN
 F 2 "" H 7550 3000 60  0000 C CNN
@@
 Connection ~ 7550 3600
 $Comp
-L +5V #PWR?
+L +5V #PWR062
 U 1 1 56AE9B39
 P 7900 3000
-F 0 "#PWR?" H 7900 3090 20  0001 C CNN
+F 0 "#PWR062" H 7900 3090 20  0001 C CNN
 F 1 "+5V" H 7900 3090 30  0000 C CNN
 F 2 "" H 7900 3000 60  0000 C CNN
@@
 Text HLabel 8050 4000 2    60   Output ~ 0
 10Hz
-$Comp
-L GND #PWR?
-U 1 1 56AE9DDF
-P 7850 3900
-F 0 "#PWR?" H 7850 3900 30  0001 C CNN
-F 1 "GND" H 7850 3830 30  0001 C CNN
-F 2 "" H 7850 3900 60  0000 C CNN
-F 3 "" H 7850 3900 60  0000 C CNN
-	1    7850 3900
-	0    1    1    0
-$EndComp
-Wire Wire Line
-	8050 3900 7850 3900
 Wire Notes Line
 	8000 3700 8000 4100
@@
 	5700 4700 5700 3700
 Wire Wire Line
-	8050 4000 7550 4000
+	7550 4000 8050 4000
 Connection ~ 7550 4000
 $Comp
-L USR R?
+L USR R26
 U 1 1 56AEA0D0
 P 7850 4300
-F 0 "R?" V 7930 4300 40  0000 C CNN
+F 0 "R26" V 7930 4300 40  0000 C CNN
 F 1 "1K" V 7750 4300 40  0000 C CNN
 F 2 "~" V 7780 4300 30  0000 C CNN
@@
 Connection ~ 7850 4000
 $Comp
-L LED D?
+L LED D23
 U 1 1 56AEA10C
 P 7850 4800
-F 0 "D?" H 7850 4900 50  0000 C CNN
+F 0 "D23" H 7850 4900 50  0000 C CNN
 F 1 "LED" H 7850 4700 50  0000 C CNN
 F 2 "~" H 7850 4800 60  0000 C CNN
@@
 Wire Wire Line
 	7850 4550 7850 4600
-$Comp
-L GND #PWR?
-U 1 1 56AEA186
-P 7850 5200
-F 0 "#PWR?" H 7850 5200 30  0001 C CNN
-F 1 "GND" H 7850 5130 30  0001 C CNN
-F 2 "" H 7850 5200 60  0000 C CNN
-F 3 "" H 7850 5200 60  0000 C CNN
-	1    7850 5200
-	1    0    0    -1
-$EndComp
-Wire Wire Line
-	7850 5000 7850 5200
-$Comp
-L DIODE D?
+Wire Wire Line
+	7850 5200 7850 5000
+$Comp
+L DIODE D22
 U 1 1 56CBDB3C
 P 4600 3950
-F 0 "D?" H 4600 4050 40  0000 C CNN
+F 0 "D22" H 4600 4050 40  0000 C CNN
 F 1 "DIODE" H 4600 3850 40  0001 C CNN
 F 2 "~" H 4600 3950 60  0000 C CNN
@@
 $EndComp
 $Comp
-L DIODE D?
+L DIODE D19
 U 1 1 56CBDB42
 P 4600 3650
-F 0 "D?" H 4600 3750 40  0000 C CNN
+F 0 "D19" H 4600 3750 40  0000 C CNN
 F 1 "DIODE" H 4600 3550 40  0001 C CNN
 F 2 "~" H 4600 3650 60  0000 C CNN
@@
 $EndComp
 $Comp
-L DIODE D?
+L DIODE D18
 U 1 1 56CBDB48
 P 3900 3650
-F 0 "D?" H 3900 3750 40  0000 C CNN
+F 0 "D18" H 3900 3750 40  0000 C CNN
 F 1 "DIODE" H 3900 3550 40  0001 C CNN
 F 2 "~" H 3900 3650 60  0000 C CNN
@@
 $EndComp
 $Comp
-L DIODE D?
+L DIODE D21
 U 1 1 56CBDB4E
 P 3900 3950
-F 0 "D?" H 3900 4050 40  0000 C CNN
+F 0 "D21" H 3900 4050 40  0000 C CNN
 F 1 "DIODE" H 3900 3850 40  0001 C CNN
 F 2 "~" H 3900 3950 60  0000 C CNN
@@
 Connection ~ 4100 3950
 Connection ~ 3700 3650
+$Comp
+L USR R24
+U 1 1 574C8025
+P 2900 3800
+F 0 "R24" V 2980 3800 40  0000 C CNN
+F 1 "0" V 2800 3800 40  0000 C CNN
+F 2 "~" V 2830 3800 30  0000 C CNN
+F 3 "~" H 2900 3800 30  0000 C CNN
+	1    2900 3800
+	1    0    0    -1
+$EndComp
+Wire Wire Line
+	2900 4050 2900 4350
+Connection ~ 2900 4300
+Wire Wire Line
+	2900 5200 7850 5200
+Connection ~ 6300 5200
+Connection ~ 5300 5200
+Connection ~ 4800 5200
+Connection ~ 3300 5200
+$Comp
+L USGND #PWR063
+U 1 1 574C81EB
+P 5300 5250
+F 0 "#PWR063" H 5300 5250 30  0001 C CNN
+F 1 "USGND" H 5300 5180 30  0001 C CNN
+F 2 "~" H 5300 5250 60  0000 C CNN
+F 3 "~" H 5300 5250 60  0000 C CNN
+	1    5300 5250
+	1    0    0    -1
+$EndComp
+$Comp
+L USGND #PWR064
+U 1 1 574C83DC
+P 7950 3900
+F 0 "#PWR064" H 7950 3900 30  0001 C CNN
+F 1 "USGND" H 7950 3830 30  0001 C CNN
+F 2 "~" H 7950 3900 60  0000 C CNN
+F 3 "~" H 7950 3900 60  0000 C CNN
+	1    7950 3900
+	0    1    1    0
+$EndComp
+Wire Wire Line
+	7950 3900 8050 3900
+Wire Wire Line
+	2900 3550 2900 3400
 $EndSCHEMATC
