File: schematic/power-board.sch (KiCad schematic (older format))
At the start: 17 parts, among them U7 4040, U8 7805

Commit message: passes ERC
Parts:
- renumbered C9 to C31, C10 to C32, C11 to C33, D17 to D38, D18 to D39, D19 to D40, D20 to D41, D21 to D42, D22 to D43, D23 to D44, R22 to R37, R23 to R38, R24 to R39, R25 to R40, R26 to R41, U7 to U26, U8 to U27
Changed lines of the file:
@@
 	3700 3650 3700 4300
 $Comp
-L CP1 C9
+L CP1 C31
 U 1 1 56AE939E
 P 4300 4300
-F 0 "C9" H 4350 4400 50  0000 L CNN
+F 0 "C31" H 4350 4400 50  0000 L CNN
 F 1 "220uF" H 4350 4200 50  0000 L CNN
 F 2 "~" H 4300 4300 60  0000 C CNN
@@
 Connection ~ 3700 3950
 $Comp
-L 7805 U8
+L 7805 U27
 U 1 1 56AE9417
 P 3300 4350
-F 0 "U8" H 3450 4154 60  0000 C CNN
+F 0 "U27" H 3450 4154 60  0000 C CNN
 F 1 "7805" H 3300 4550 60  0000 C CNN
 F 2 "" H 3300 4350 60  0000 C CNN
@@
 	3300 4600 3300 5200
 $Comp
-L CSMALL C10
+L CSMALL C32
 U 1 1 56AE9499
 P 2900 4450
-F 0 "C10" H 2925 4500 30  0000 L CNN
+F 0 "C32" H 2925 4500 30  0000 L CNN
 F 1 "1uF" H 2925 4400 30  0000 L CNN
 F 2 "~" H 2900 4450 60  0000 C CNN
@@
 	2900 4550 2900 5200
 $Comp
-L +5V #PWR058
+L +5V #PWR0134
 U 1 1 56AE94DA
 P 2900 3400
-F 0 "#PWR058" H 2900 3490 20  0001 C CNN
+F 0 "#PWR0134" H 2900 3490 20  0001 C CNN
 F 1 "+5V" H 2900 3490 30  0000 C CNN
 F 2 "" H 2900 3400 60  0000 C CNN
@@
 	4400 3000 4100 3000
 $Comp
-L 4040 U7
+L 4040 U26
 U 1 1 56AE9575
 P 6350 3950
-F 0 "U7" H 6450 4600 60  0000 C CNN
+F 0 "U26" H 6450 4600 60  0000 C CNN
 F 1 "4040" H 6600 3300 60  0000 C CNN
 F 2 "" H 6350 3950 60  0000 C CNN
@@
 Connection ~ 4300 3400
 $Comp
-L USR R23
+L USR R38
 U 1 1 56AE976F
 P 5050 3400
-F 0 "R23" V 5130 3400 40  0000 C CNN
+F 0 "R38" V 5130 3400 40  0000 C CNN
 F 1 "2K7" V 4950 3400 40  0000 C CNN
 F 2 "~" V 4980 3400 30  0000 C CNN
@@
 Connection ~ 4800 3400
 $Comp
-L USR R25
+L USR R40
 U 1 1 56AE9781
 P 5300 3950
-F 0 "R25" V 5380 3950 40  0000 C CNN
+F 0 "R40" V 5380 3950 40  0000 C CNN
 F 1 "1K" V 5200 3950 40  0000 C CNN
 F 2 "~" V 5230 3950 30  0000 C CNN
@@
 	5300 3400 5700 3400
 $Comp
-L CSMALL C11
+L CSMALL C33
 U 1 1 56AE9894
 P 6300 5050
-F 0 "C11" H 6325 5100 30  0000 L CNN
+F 0 "C33" H 6325 5100 30  0000 L CNN
 F 1 "100nF BYPASS" H 6325 5000 30  0000 L CNN
 F 2 "~" H 6300 5050 60  0000 C CNN
@@
 $EndComp
 $Comp
-L +5V #PWR059
+L +5V #PWR0135
 U 1 1 56AE98AF
 P 6300 4900
-F 0 "#PWR059" H 6300 4990 20  0001 C CNN
+F 0 "#PWR0135" H 6300 4990 20  0001 C CNN
 F 1 "+5V" H 6300 4990 30  0000 C CNN
 F 2 "" H 6300 4900 60  0000 C CNN
@@
 NoConn ~ 7000 4500
 $Comp
-L DIODE D17
+L DIODE D38
 U 1 1 56AE9A06
 P 7350 3600
-F 0 "D17" H 7350 3700 40  0000 C CNN
+F 0 "D38" H 7350 3700 40  0000 C CNN
 F 1 "DIODE" H 7350 3500 40  0001 C CNN
 F 2 "~" H 7350 3600 60  0000 C CNN
@@
 $EndComp
 $Comp
-L DIODE D20
+L DIODE D41
 U 1 1 56AE9A11
 P 7350 3750
-F 0 "D20" H 7350 3850 40  0000 C CNN
+F 0 "D41" H 7350 3850 40  0000 C CNN
 F 1 "DIODE" H 7350 3650 40  0001 C CNN
 F 2 "~" H 7350 3750 60  0000 C CNN
@@
 Connection ~ 7550 3750
 $Comp
-L USR R22
+L USR R37
 U 1 1 56AE9AD5
 P 7550 3300
-F 0 "R22" V 7630 3300 40  0000 C CNN
+F 0 "R37" V 7630 3300 40  0000 C CNN
 F 1 "100K" V 7450 3300 40  0000 C CNN
 F 2 "~" V 7480 3300 30  0000 C CNN
@@
 $EndComp
 $Comp
-L +5V #PWR060
+L +5V #PWR0136
 U 1 1 56AE9ADB
 P 7550 3000
-F 0 "#PWR060" H 7550 3090 20  0001 C CNN
+F 0 "#PWR0136" H 7550 3090 20  0001 C CNN
 F 1 "+5V" H 7550 3090 30  0000 C CNN
 F 2 "" H 7550 3000 60  0000 C CNN
@@
 Connection ~ 7550 3600
 $Comp
-L +5V #PWR061
+L +5V #PWR0137
 U 1 1 56AE9B39
 P 7900 3000
-F 0 "#PWR061" H 7900 3090 20  0001 C CNN
+F 0 "#PWR0137" H 7900 3090 20  0001 C CNN
 F 1 "+5V" H 7900 3090 30  0000 C CNN
 F 2 "" H 7900 3000 60  0000 C CNN
@@
 Connection ~ 7550 4000
 $Comp
-L USR R26
+L USR R41
 U 1 1 56AEA0D0
 P 7850 4300
-F 0 "R26" V 7930 4300 40  0000 C CNN
+F 0 "R41" V 7930 4300 40  0000 C CNN
 F 1 "1K" V 7750 4300 40  0000 C CNN
 F 2 "~" V 7780 4300 30  0000 C CNN
@@
 Connection ~ 7850 4000
 $Comp
-L LED D23
+L LED D44
 U 1 1 56AEA10C
 P 7850 4800
-F 0 "D23" H 7850 4900 50  0000 C CNN
+F 0 "D44" H 7850 4900 50  0000 C CNN
 F 1 "LED" H 7850 4700 50  0000 C CNN
 F 2 "~" H 7850 4800 60  0000 C CNN
@@
 	7850 5200 7850 5000
 $Comp
-L DIODE D22
+L DIODE D43
 U 1 1 56CBDB3C
 P 4600 3950
-F 0 "D22" H 4600 4050 40  0000 C CNN
+F 0 "D43" H 4600 4050 40  0000 C CNN
 F 1 "DIODE" H 4600 3850 40  0001 C CNN
 F 2 "~" H 4600 3950 60  0000 C CNN
@@
 $EndComp
 $Comp
-L DIODE D19
+L DIODE D40
 U 1 1 56CBDB42
 P 4600 3650
-F 0 "D19" H 4600 3750 40  0000 C CNN
+F 0 "D40" H 4600 3750 40  0000 C CNN
 F 1 "DIODE" H 4600 3550 40  0001 C CNN
 F 2 "~" H 4600 3650 60  0000 C CNN
@@
 $EndComp
 $Comp
-L DIODE D18
+L DIODE D39
 U 1 1 56CBDB48
 P 3900 3650
-F 0 "D18" H 3900 3750 40  0000 C CNN
+F 0 "D39" H 3900 3750 40  0000 C CNN
 F 1 "DIODE" H 3900 3550 40  0001 C CNN
 F 2 "~" H 3900 3650 60  0000 C CNN
@@
 $EndComp
 $Comp
-L DIODE D21
+L DIODE D42
 U 1 1 56CBDB4E
 P 3900 3950
-F 0 "D21" H 3900 4050 40  0000 C CNN
+F 0 "D42" H 3900 4050 40  0000 C CNN
 F 1 "DIODE" H 3900 3850 40  0001 C CNN
 F 2 "~" H 3900 3950 60  0000 C CNN
@@
 Connection ~ 3700 3650
 $Comp
-L USR R24
+L USR R39
 U 1 1 574C8025
 P 2900 3800
-F 0 "R24" V 2980 3800 40  0000 C CNN
+F 0 "R39" V 2980 3800 40  0000 C CNN
 F 1 "0" V 2800 3800 40  0000 C CNN
 F 2 "~" V 2830 3800 30  0000 C CNN
@@
 Connection ~ 3300 5200
 $Comp
-L USGND #PWR062
+L USGND #PWR0138
 U 1 1 574C81EB
 P 5300 5250
-F 0 "#PWR062" H 5300 5250 30  0001 C CNN
+F 0 "#PWR0138" H 5300 5250 30  0001 C CNN
 F 1 "USGND" H 5300 5180 30  0001 C CNN
 F 2 "~" H 5300 5250 60  0000 C CNN
@@
 $EndComp
 $Comp
-L USGND #PWR063
+L USGND #PWR0139
 U 1 1 574C83DC
 P 7950 3900
-F 0 "#PWR063" H 7950 3900 30  0001 C CNN
+F 0 "#PWR0139" H 7950 3900 30  0001 C CNN
 F 1 "USGND" H 7950 3830 30  0001 C CNN
 F 2 "~" H 7950 3900 60  0000 C CNN
