File: schematic/logic-board.sch (KiCad schematic (older format))
At the start: 51 parts

Commit message: one more digit
Parts:
- added D? (x8): DIODE, ~, symbol DIODE
- added Q?: ZVN4206, ~, symbol MOSFET_N
- added R? (x4): 10K, ~, symbol USR
- added R? (x2): 100K, ~, symbol USR
Connections:
- wire segments 87 -> 101

Commit message: schematic matches prototype
Parts:
- added D? (x2): DIODE, ~, symbol DIODE
- added P?: 2-PIN_HEADER, ~, symbol 2-PIN_HEADER
- added Q?: ZVN4206, ~, symbol MOSFET_N
- added R?: 10K, ~, symbol USR
- added R?: 100K, ~, symbol USR
- added U? (x2): 4013, symbol 4013
Connections:
- net labels added: AM, TEN-HOURS
- wire segments 101 -> 131
Other:
- note added: "RESET"
- moved on the sheet: D?

Commit message: ok now it is correct mostly
Parts:
- added D?: DIODE, ~, symbol DIODE
- added R?: 100K, ~, symbol USR
Connections:
- wire segments 131 -> 134
Other:
- note added: "NOR"
Changed lines of the file:
@@
 Connection ~ 7650 12900
 Wire Wire Line
-	7200 12900 7200 13100
+	7200 12600 7200 13100
 Connection ~ 7750 12550
 $Comp
@@
 $EndComp
 Connection ~ 6400 14050
-Text Notes 7400 10600 0    60   ~ 0
+Text Notes 7300 11800 1    60   ~ 0
 RESET
 $Comp
@@
 	7600 7400 7600 8150
 Connection ~ 6900 13300
+$Comp
+L USR R?
+U 1 1 57B150E2
+P 6400 12600
+F 0 "R?" V 6480 12600 40  0000 C CNN
+F 1 "100K" V 6300 12600 40  0000 C CNN
+F 2 "~" V 6330 12600 30  0000 C CNN
+F 3 "~" H 6400 12600 30  0000 C CNN
+	1    6400 12600
+	0    1    1    0
+$EndComp
+$Comp
+L GND #PWR?
+U 1 1 57B150E8
+P 6150 12600
+F 0 "#PWR?" H 6150 12600 30  0001 C CNN
+F 1 "GND" H 6150 12530 30  0001 C CNN
+F 2 "" H 6150 12600 60  0000 C CNN
+F 3 "" H 6150 12600 60  0000 C CNN
+	1    6150 12600
+	0    1    1    0
+$EndComp
+Connection ~ 6150 12600
+Wire Wire Line
+	6650 12600 7200 12600
+Connection ~ 7200 12900
+$Comp
+L DIODE D?
+U 1 1 57B1533C
+P 6650 11550
+F 0 "D?" H 6650 11650 40  0000 C CNN
+F 1 "DIODE" H 6650 11450 40  0001 C CNN
+F 2 "~" H 6650 11550 60  0000 C CNN
+F 3 "~" H 6650 11550 60  0000 C CNN
+	1    6650 11550
+	0    1    1    0
+$EndComp
+Wire Wire Line
+	6650 11250 6650 11350
+Connection ~ 6650 11250
+Wire Wire Line
+	6650 11750 6650 12600
+Text Notes 6800 13100 1    60   ~ 0
+NOR
 $EndSCHEMATC

Commit message: added shift registers
Parts:
- added P?: 3-PIN_HEADER, ~, symbol 3-PIN_HEADER
- added U? (x2): 4094, ~, symbol 4094
Connections:
- net labels added: CLOCK, DATA, SET
- wire segments 134 -> 154
- no-connect marks 3 -> 6
Changed lines of the file:
@@
 Text Notes 6800 13100 1    60   ~ 0
 NOR
+$Comp
+L 4094 U?
+U 1 1 57B161EB
+P 10800 7900
+F 0 "U?" H 11100 8350 60  0000 C CNN
+F 1 "4094" H 10450 8350 60  0000 C CNN
+F 2 "~" H 10750 7700 60  0000 C CNN
+F 3 "~" H 10750 7700 60  0000 C CNN
+	1    10800 7900
+	1    0    0    -1
+$EndComp
+$Comp
+L 4094 U?
+U 1 1 57B161F8
+P 12750 7900
+F 0 "U?" H 13050 8350 60  0000 C CNN
+F 1 "4094" H 12400 8350 60  0000 C CNN
+F 2 "~" H 12700 7700 60  0000 C CNN
+F 3 "~" H 12700 7700 60  0000 C CNN
+	1    12750 7900
+	1    0    0    -1
+$EndComp
+Wire Wire Line
+	7000 8550 7000 8250
+$Comp
+L 3-PIN_HEADER P?
+U 1 1 57B167C1
+P 9250 7700
+F 0 "P?" H 8950 7700 50  0000 C CNN
+F 1 "3-PIN_HEADER" H 9250 7900 50  0001 C CNN
+F 2 "~" H 9300 7850 60  0000 C CNN
+F 3 "~" H 9300 7850 60  0000 C CNN
+	1    9250 7700
+	0    -1   1    0
+$EndComp
+Text HLabel 9200 7600 0    60   Input ~ 0
+DATA
+Text HLabel 9200 7700 0    60   Input ~ 0
+CLOCK
+Text HLabel 9200 7800 0    60   Input ~ 0
+SET
+Wire Notes Line
+	9200 7500 8800 7500
+Wire Notes Line
+	8800 7500 8800 7900
+Wire Notes Line
+	8800 7900 9200 7900
+Wire Wire Line
+	9200 7600 10050 7600
+Wire Wire Line
+	9200 7700 10050 7700
+Wire Wire Line
+	9200 7800 10050 7800
+Wire Wire Line
+	10050 7800 10050 8000
+Connection ~ 10050 7850
+$Comp
+L +5V #PWR?
+U 1 1 57B17010
+P 11550 7900
+F 0 "#PWR?" H 11550 7990 20  0001 C CNN
+F 1 "+5V" H 11550 7990 30  0000 C CNN
+F 2 "" H 11550 7900 60  0000 C CNN
+F 3 "" H 11550 7900 60  0000 C CNN
+	1    11550 7900
+	0    1    1    0
+$EndComp
+Connection ~ 11550 7900
+$Comp
+L GND #PWR?
+U 1 1 57B1701F
+P 11550 8000
+F 0 "#PWR?" H 11550 8000 30  0001 C CNN
+F 1 "GND" H 11550 7930 30  0001 C CNN
+F 2 "" H 11550 8000 60  0000 C CNN
+F 3 "" H 11550 8000 60  0000 C CNN
+	1    11550 8000
+	0    -1   -1   0
+$EndComp
+Connection ~ 11550 8000
+Connection ~ 9500 7600
+Connection ~ 9500 7700
+Connection ~ 9500 7800
+Text GLabel 9750 7900 3    60   Output ~ 0
+SET
+Wire Wire Line
+	9750 7900 9750 7800
+Connection ~ 9750 7800
+Text GLabel 8600 10550 1    60   Input ~ 0
+SET
+Wire Wire Line
+	8600 10550 8600 10850
+Text GLabel 10300 10550 1    60   Input ~ 0
+SET
+Wire Wire Line
+	10300 10550 10300 10850
+Text GLabel 12250 11150 1    60   Input ~ 0
+SET
+Wire Wire Line
+	12250 11150 12250 11250
+Text GLabel 13600 10750 1    60   Input ~ 0
+SET
+Wire Wire Line
+	13600 10750 13600 10850
+Text GLabel 14550 10350 1    60   Input ~ 0
+SET
+Wire Wire Line
+	14550 10350 14550 10650
+Text GLabel 16150 10350 1    60   Input ~ 0
+SET
+Wire Wire Line
+	16150 10350 16150 10650
+Wire Wire Line
+	11550 7700 11750 7700
+Wire Wire Line
+	11750 7700 11750 7600
+Wire Wire Line
+	11750 7600 12000 7600
+Wire Wire Line
+	9900 7700 9900 7300
+Wire Wire Line
+	9900 7300 11900 7300
+Wire Wire Line
+	11900 7300 11900 7700
+Wire Wire Line
+	11900 7700 12000 7700
+Connection ~ 9900 7700
+NoConn ~ 11550 7600
+NoConn ~ 13500 7600
+NoConn ~ 13500 7700
+$Comp
+L +5V #PWR?
+U 1 1 57B1805F
+P 13500 7900
+F 0 "#PWR?" H 13500 7990 20  0001 C CNN
+F 1 "+5V" H 13500 7990 30  0000 C CNN
+F 2 "" H 13500 7900 60  0000 C CNN
+F 3 "" H 13500 7900 60  0000 C CNN
+	1    13500 7900
+	0    1    1    0
+$EndComp
+Connection ~ 13500 7900
+$Comp
+L GND #PWR?
+U 1 1 57B18065
+P 13500 8000
+F 0 "#PWR?" H 13500 8000 30  0001 C CNN
+F 1 "GND" H 13500 7930 30  0001 C CNN
+F 2 "" H 13500 8000 60  0000 C CNN
+F 3 "" H 13500 8000 60  0000 C CNN
+	1    13500 8000
+	0    -1   -1   0
+$EndComp
+Connection ~ 13500 8000
+Text GLabel 12000 8100 3    60   Input ~ 0
+SET
+Wire Wire Line
+	12000 7850 12000 8100
+Connection ~ 12000 8000
 $EndSCHEMATC

Commit message: ok i think this should be hooked up right
Parts:
- added D? (x2): DIODE, ~, symbol DIODE
- added R? (x2): 100K, ~, symbol USR
- added R?: 10K, ~, symbol USR
- added RR? (x2): 100K, ~, symbol RR8
Connections:
- wire segments 154 -> 206
Other:
- moved on the sheet: R?

Commit message: resized page
Connections:
- wire segments 206 -> 203
Other:
- note added: "0121234567890121234..."
- moved on the sheet: D?, R?, U?A, U?B

Commit message: 1st digit bug fix, disabled TX zeros
Parts:
- removed D? (x2): DIODE, ~, symbol DIODE
- removed R?: 100K, ~, symbol USR
Connections:
- wire segments 203 -> 200
Changed lines of the file:
@@
 Sheet 5 5
 Title "LOGIC CLOCK LOGIC BOARD"
-Date "15 aug 2016"
+Date "23 aug 2016"
 Rev "1"
 Comp "Michael Craft"
@@
 F 3 "" H 13150 5200 60  0000 C CNN
 	1    13150 5200
-	0    -1   -1   0
-$EndComp
-$Comp
-L DIODE D?
-U 1 1 57893821
-P 14250 5000
-F 0 "D?" H 14250 5100 40  0000 C CNN
-F 1 "DIODE" H 14250 4900 40  0001 C CNN
-F 2 "~" H 14250 5000 60  0000 C CNN
-F 3 "~" H 14250 5000 60  0000 C CNN
-	1    14250 5000
-	0    1    1    0
-$EndComp
-$Comp
-L DIODE D?
-U 1 1 57893827
-P 14150 5000
-F 0 "D?" H 14150 5100 40  0000 C CNN
-F 1 "DIODE" H 14150 4900 40  0001 C CNN
-F 2 "~" H 14150 5000 60  0000 C CNN
-F 3 "~" H 14150 5000 60  0000 C CNN
-	1    14150 5000
-	0    1    1    0
-$EndComp
-$Comp
-L USR R?
-U 1 1 5789382D
-P 14500 5200
-F 0 "R?" V 14580 5200 40  0000 C CNN
-F 1 "100K" V 14400 5200 40  0000 C CNN
-F 2 "~" V 14430 5200 30  0000 C CNN
-F 3 "~" H 14500 5200 30  0000 C CNN
-	1    14500 5200
-	0    1    1    0
-$EndComp
-$Comp
-L GND #PWR?
-U 1 1 57893834
-P 14750 5200
-F 0 "#PWR?" H 14750 5200 30  0001 C CNN
-F 1 "GND" H 14750 5130 30  0001 C CNN
-F 2 "" H 14750 5200 60  0000 C CNN
-F 3 "" H 14750 5200 60  0000 C CNN
-	1    14750 5200
 	0    -1   -1   0
 $EndComp
@@
 Text GLabel 12550 4500 1    60   Input ~ 0
 SET
-Text GLabel 14150 4500 1    60   Input ~ 0
+Text GLabel 14200 5050 1    60   Input ~ 0
 SET
 NoConn ~ 9550 1450
@@
 	12600 5200 12600 5400
 Connection ~ 12600 5200
-Connection ~ 14250 5200
-Connection ~ 14750 5200
-Wire Wire Line
-	14150 5200 14250 5200
-Wire Wire Line
-	14200 5200 14200 5400
-Connection ~ 14200 5200
 Connection ~ 11700 5400
 Connection ~ 12200 5400
@@
 Wire Wire Line
 	12500 4700 12500 5400
-Wire Wire Line
-	14250 4800 14250 4700
-Connection ~ 14250 4700
 Wire Wire Line
 	13450 4600 13450 6600
@@
 Wire Wire Line
 	12550 4500 12550 4800
-Wire Wire Line
-	14150 4500 14150 4800
 Wire Wire Line
 	9550 1550 9750 1550
@@
 Text Notes 4000 9750 0    60   ~ 0
 0121234567890121234...
+Wire Wire Line
+	14200 5050 14200 5400
 $EndSCHEMATC

Commit message: 2nd digit bug fix
Parts:
- removed D? (x2): DIODE, ~, symbol DIODE
- removed R?: 100K, ~, symbol USR
Connections:
- wire segments 200 -> 197
Changed lines of the file:
@@
-$Comp
-L DIODE D?
-U 1 1 578936D7
-P 12650 5000
-F 0 "D?" H 12650 5100 40  0000 C CNN
-F 1 "DIODE" H 12650 4900 40  0001 C CNN
-F 2 "~" H 12650 5000 60  0000 C CNN
-F 3 "~" H 12650 5000 60  0000 C CNN
-	1    12650 5000
-	0    1    1    0
-$EndComp
-$Comp
-L DIODE D?
-U 1 1 578936DD
-P 12550 5000
-F 0 "D?" H 12550 5100 40  0000 C CNN
-F 1 "DIODE" H 12550 4900 40  0001 C CNN
-F 2 "~" H 12550 5000 60  0000 C CNN
-F 3 "~" H 12550 5000 60  0000 C CNN
-	1    12550 5000
-	0    1    1    0
-$EndComp
-$Comp
-L USR R?
-U 1 1 5789377D
-P 12900 5200
-F 0 "R?" V 12980 5200 40  0000 C CNN
-F 1 "100K" V 12800 5200 40  0000 C CNN
-F 2 "~" V 12830 5200 30  0000 C CNN
-F 3 "~" H 12900 5200 30  0000 C CNN
-	1    12900 5200
-	0    1    1    0
-$EndComp
-$Comp
-L GND #PWR?
-U 1 1 57893785
-P 13150 5200
-F 0 "#PWR?" H 13150 5200 30  0001 C CNN
-F 1 "GND" H 13150 5130 30  0001 C CNN
-F 2 "" H 13150 5200 60  0000 C CNN
-F 3 "" H 13150 5200 60  0000 C CNN
-	1    13150 5200
-	0    -1   -1   0
-$EndComp
 $Comp
 L DIODE D?
@@
 Text GLabel 11600 4900 1    60   Input ~ 0
 SET
-Text GLabel 12550 4500 1    60   Input ~ 0
+Text GLabel 12600 5050 1    60   Input ~ 0
 SET
 Text GLabel 14200 5050 1    60   Input ~ 0
@@
 	10650 4600 10650 5400
 Connection ~ 11300 5400
-Connection ~ 12650 5200
-Connection ~ 13150 5200
-Wire Wire Line
-	12550 5200 12650 5200
-Wire Wire Line
-	12600 5200 12600 5400
-Connection ~ 12600 5200
 Connection ~ 11700 5400
 Connection ~ 12200 5400
@@
 	10650 4600 13450 4600
 Connection ~ 13450 5200
-Wire Wire Line
-	12650 4600 12650 4800
-Connection ~ 12650 4600
 Connection ~ 11200 6600
 Connection ~ 11300 6600
@@
 Wire Wire Line
 	11600 4900 11600 5000
-Wire Wire Line
-	12550 4500 12550 4800
 Wire Wire Line
 	9550 1550 9750 1550
@@
 Wire Wire Line
 	14200 5050 14200 5400
+Wire Wire Line
+	12600 5050 12600 5400
 $EndSCHEMATC
