File: schematic/logic-board.sch (KiCad schematic (older format))
At the start: 82 parts

Commit message: added some resistors, works better
Parts:
- added R? (x2): 10K, ~, symbol USR
Connections:
- wire segments 202 -> 203
Changed lines of the file:
@@
 Connection ~ 11950 6950
 Wire Wire Line
-	12300 5550 11750 5550
-Wire Wire Line
-	11750 5550 11750 6750
-Wire Wire Line
-	11750 6750 11450 6750
+	11450 6750 11850 6750
 Connection ~ 11450 6900
 Connection ~ 9900 5400
@@
 Connection ~ 5750 6700
 Connection ~ 4850 6450
-Wire Wire Line
-	5100 4800 6700 4800
-Wire Wire Line
-	6700 4800 6700 5000
 Connection ~ 5350 6450
 Connection ~ 4900 8200
@@
 Wire Wire Line
 	5100 4450 5100 4800
-Connection ~ 5350 4800
 Wire Wire Line
 	5350 4800 5350 6700
@@
 Wire Wire Line
 	8550 6750 8550 6300
+Wire Wire Line
+	5100 4800 6200 4800
+$Comp
+L USR R?
+U 1 1 5831FE53
+P 6450 4800
+F 0 "R?" V 6530 4800 40  0000 C CNN
+F 1 "10K" V 6350 4800 40  0000 C CNN
+F 2 "~" V 6380 4800 30  0000 C CNN
+F 3 "~" H 6450 4800 30  0000 C CNN
+	1    6450 4800
+	0    1    1    0
+$EndComp
+Wire Wire Line
+	6700 4800 6700 5000
+Connection ~ 5350 4800
+$Comp
+L USR R?
+U 1 1 5832017A
+P 11850 6000
+F 0 "R?" V 11930 6000 40  0000 C CNN
+F 1 "10K" V 11750 6000 40  0000 C CNN
+F 2 "~" V 11780 6000 30  0000 C CNN
+F 3 "~" H 11850 6000 30  0000 C CNN
+	1    11850 6000
+	1    0    0    -1
+$EndComp
+Wire Wire Line
+	12300 5550 11850 5550
+Wire Wire Line
+	11850 5550 11850 5750
+Wire Wire Line
+	11850 6750 11850 6250
 $EndSCHEMATC

Commit message: replaced some diode gates with CMOS gates
Parts:
- removed D? (x6): DIODE, ~, symbol DIODE
- removed R? (x3): 100K, ~, symbol USR
- removed R? (x3): 10K, ~, symbol USR
- added U? (x3): 4071, symbol 4071
Connections:
- net labels added: TEN-MIN_CARRY
- wire segments 203 -> 199

Commit message: idk what changed i hope nothing is broken
Parts:
- removed D? (x11): DIODE, ~, symbol DIODE
- removed Q? (x2): ZVN4206, ~, symbol MOSFET_N
- removed R? (x5): 10K, ~, symbol USR
- removed R? (x4): 100K, ~, symbol USR
- added U? (x3): 4071, symbol 4071
- added U? (x2): 4072, symbol 4072
- added U? (x2): 4584, ~, symbol 4584
Connections:
- wire segments 199 -> 204

Commit message: prototype works!
Parts:
- removed D? (x2): DIODE, ~, symbol DIODE
- removed R?: 47K, ~, symbol USR
- added U?: 4081, symbol 4081
Connections:
- wire segments 204 -> 207
Changed lines of the file:
@@
 Sheet 5 8
 Title "LOGIC CLOCK LOGIC BOARD"
-Date "30 oct 2018"
+Date "19 nov 2018"
 Rev "1"
 Comp "Michael Craft"
@@
 	-1   0    0    1
 $EndComp
-$Comp
-L DIODE D?
-U 1 1 578978A8
-P 5550 6700
-F 0 "D?" H 5550 6800 40  0000 C CNN
-F 1 "DIODE" H 5550 6600 40  0001 C CNN
-F 2 "~" H 5550 6700 60  0000 C CNN
-F 3 "~" H 5550 6700 60  0000 C CNN
-	1    5550 6700
-	1    0    0    1
-$EndComp
-$Comp
-L DIODE D?
-U 1 1 57897C09
-P 5150 5400
-F 0 "D?" H 5150 5500 40  0000 C CNN
-F 1 "DIODE" H 5150 5300 40  0001 C CNN
-F 2 "~" H 5150 5400 60  0000 C CNN
-F 3 "~" H 5150 5400 60  0000 C CNN
-	1    5150 5400
-	-1   0    0    1
-$EndComp
-$Comp
-L USR R?
-U 1 1 57897CFB
-P 5100 6450
-F 0 "R?" V 5180 6450 40  0000 C CNN
-F 1 "47K" V 5000 6450 40  0000 C CNN
-F 2 "~" V 5030 6450 30  0000 C CNN
-F 3 "~" H 5100 6450 30  0000 C CNN
-	1    5100 6450
-	0    1    1    0
-$EndComp
-$Comp
-L +5V #PWR?
-U 1 1 57897D01
-P 4850 6450
-F 0 "#PWR?" H 4850 6540 20  0001 C CNN
-F 1 "+5V" H 4850 6540 30  0000 C CNN
-F 2 "" H 4850 6450 60  0000 C CNN
-F 3 "" H 4850 6450 60  0000 C CNN
-	1    4850 6450
-	0    -1   -1   0
-$EndComp
-Text Notes 5300 5950 1    60   ~ 0
+Text Notes 5400 6150 1    60   ~ 0
 RESET
 $Comp
@@
 	5750 6600 5750 7900
 Connection ~ 6300 5400
-Connection ~ 5750 6700
-Connection ~ 4850 6450
-Connection ~ 5350 6450
-Connection ~ 5350 5400
-Wire Wire Line
-	4050 5400 4950 5400
-Connection ~ 5350 6150
 Wire Wire Line
 	4300 4850 4300 5800
@@
 Wire Wire Line
 	4200 1650 6200 1650
-Connection ~ 4400 5400
 Wire Wire Line
 	1300 7450 1300 1550
@@
 Wire Wire Line
 	4650 5400 4650 6850
-Connection ~ 4650 5400
 Wire Wire Line
 	5000 2700 5000 2400
@@
 	5800 3250 5800 5400
 Wire Wire Line
-	5350 6150 4350 6150
-Wire Wire Line
 	4300 4850 2850 4850
 Wire Wire Line
@@
 	12600 5050 12600 5400
 Wire Wire Line
-	5100 4450 5100 4800
-Wire Wire Line
-	5350 4800 5350 6700
+	5100 4450 5100 5400
 Wire Wire Line
 	15050 4150 15050 6600
@@
 Connection ~ 8150 7000
 Wire Wire Line
-	5100 4800 5350 4800
-Wire Wire Line
 	5650 5350 5650 5400
 Wire Wire Line
@@
 Wire Wire Line
 	4350 6450 4350 6150
+$Comp
+L 4081 U?
+U 1 1 5BF34929
+P 5100 6000
+F 0 "U?" H 5100 6050 60  0000 C CNN
+F 1 "4081" H 5100 5950 60  0000 C CNN
+F 2 "" H 5100 6000 60  0000 C CNN
+F 3 "" H 5100 6000 60  0000 C CNN
+	1    5100 6000
+	0    -1   -1   0
+$EndComp
+Wire Wire Line
+	4050 5400 4650 5400
+Connection ~ 4400 5400
+Wire Wire Line
+	4650 6600 5000 6600
+Connection ~ 4650 6600
+Wire Wire Line
+	5750 6700 5200 6700
+Wire Wire Line
+	5200 6700 5200 6600
+Connection ~ 5750 6700
+Wire Wire Line
+	4350 6150 4800 6150
+Wire Wire Line
+	4800 6150 4800 4800
+Wire Wire Line
+	4800 4800 5100 4800
+Connection ~ 5100 4800
 $EndSCHEMATC

Commit message: passes ERC
Parts:
- added C16: 1uF, ~, symbol C
- added C17, C18, C19, C20, C21, C22, C23, C24, C25, C26, C27, C28, C29, C30: 100nF, ~, symbol CSMALL
- added D24: DIODE, ~, symbol DIODE
- U5: renamed from U?; symbol 4013 -> CD4013
- gave numbers to parts that had none: 51
Connections:
- wire segments 207 -> 215
Other:
- note added: "(POWER DIODE)"
- note added: "BYPASS CAPS"
- note added: "FILTER CAP"
- note added: "REVERSE POLARITY\nPROTECTION"
- moved on the sheet: D25, R29

Commit message: layout almost ready for routing
Parts:
- removed C30: 100nF, ~, symbol CSMALL
- added U? (x3): 4081, symbol 4081
Connections:
- no-connect marks 6 -> 9
Changed lines of the file:
@@
 Sheet 5 8
 Title "LOGIC CLOCK LOGIC BOARD"
-Date "19 nov 2018"
+Date "23 nov 2018"
 Rev "1"
 Comp "Michael Craft"
@@
 $EndComp
 $Comp
-L CSMALL C30
-U 1 1 5BF38085
-P 15000 2950
-F 0 "C30" H 15025 3000 30  0000 L CNN
-F 1 "100nF" H 15025 2900 30  0000 L CNN
-F 2 "~" H 15000 2950 60  0000 C CNN
-F 3 "~" H 15000 2950 60  0000 C CNN
-	1    15000 2950
-	1    0    0    -1
-$EndComp
-$Comp
 L CSMALL C24
 U 1 1 5BF3808B
@@
 	1    0    0    -1
 $EndComp
-Wire Wire Line
-	13500 2850 15000 2850
 Connection ~ 13750 2850
 Connection ~ 14000 2850
 Connection ~ 14250 2850
 Connection ~ 14500 2850
-Connection ~ 14750 2850
-Wire Wire Line
-	13500 3050 15000 3050
 Connection ~ 13750 3050
 Connection ~ 14000 3050
 Connection ~ 14250 3050
 Connection ~ 14500 3050
-Connection ~ 14750 3050
 $Comp
 L GND #PWR0132
@@
 $EndComp
 Wire Wire Line
-	14250 2800 14250 2850
+	14250 2850 14250 2800
 Text Notes 13950 2150 0    60   ~ 0
 BYPASS CAPS
+Wire Wire Line
+	13500 2850 14750 2850
+Wire Wire Line
+	13500 3050 14750 3050
+$Comp
+L 4081 U?
+U 2 1 5BF8763A
+P 1700 8600
+F 0 "U?" H 1700 8650 60  0000 C CNN
+F 1 "4081" H 1700 8550 60  0000 C CNN
+F 2 "" H 1700 8600 60  0000 C CNN
+F 3 "" H 1700 8600 60  0000 C CNN
+	2    1700 8600
+	1    0    0    -1
+$EndComp
+$Comp
+L 4081 U?
+U 3 1 5BF87645
+P 1700 9050
+F 0 "U?" H 1700 9100 60  0000 C CNN
+F 1 "4081" H 1700 9000 60  0000 C CNN
+F 2 "" H 1700 9050 60  0000 C CNN
+F 3 "" H 1700 9050 60  0000 C CNN
+	3    1700 9050
+	1    0    0    -1
+$EndComp
+$Comp
+L 4081 U?
+U 4 1 5BF87650
+P 1700 9500
+F 0 "U?" H 1700 9550 60  0000 C CNN
+F 1 "4081" H 1700 9450 60  0000 C CNN
+F 2 "" H 1700 9500 60  0000 C CNN
+F 3 "" H 1700 9500 60  0000 C CNN
+	4    1700 9500
+	1    0    0    -1
+$EndComp
+NoConn ~ 2300 8600
+NoConn ~ 2300 9050
+NoConn ~ 2300 9500
+$Comp
+L GND #PWR?
+U 1 1 5BF8765B
+P 1100 8500
+F 0 "#PWR?" H 1100 8500 30  0001 C CNN
+F 1 "GND" H 1100 8430 30  0001 C CNN
+F 2 "" H 1100 8500 60  0000 C CNN
+F 3 "" H 1100 8500 60  0000 C CNN
+	1    1100 8500
+	0    1    1    0
+$EndComp
+Connection ~ 1100 8500
+$Comp
+L GND #PWR?
+U 1 1 5BF87661
+P 1100 8700
+F 0 "#PWR?" H 1100 8700 30  0001 C CNN
+F 1 "GND" H 1100 8630 30  0001 C CNN
+F 2 "" H 1100 8700 60  0000 C CNN
+F 3 "" H 1100 8700 60  0000 C CNN
+	1    1100 8700
+	0    1    1    0
+$EndComp
+Connection ~ 1100 8700
+$Comp
+L GND #PWR?
+U 1 1 5BF87667
+P 1100 8950
+F 0 "#PWR?" H 1100 8950 30  0001 C CNN
+F 1 "GND" H 1100 8880 30  0001 C CNN
+F 2 "" H 1100 8950 60  0000 C CNN
+F 3 "" H 1100 8950 60  0000 C CNN
+	1    1100 8950
+	0    1    1    0
+$EndComp
+Connection ~ 1100 8950
+$Comp
+L GND #PWR?
+U 1 1 5BF8766D
+P 1100 9150
+F 0 "#PWR?" H 1100 9150 30  0001 C CNN
+F 1 "GND" H 1100 9080 30  0001 C CNN
+F 2 "" H 1100 9150 60  0000 C CNN
+F 3 "" H 1100 9150 60  0000 C CNN
+	1    1100 9150
+	0    1    1    0
+$EndComp
+Connection ~ 1100 9150
+$Comp
+L GND #PWR?
+U 1 1 5BF87673
+P 1100 9400
+F 0 "#PWR?" H 1100 9400 30  0001 C CNN
+F 1 "GND" H 1100 9330 30  0001 C CNN
+F 2 "" H 1100 9400 60  0000 C CNN
+F 3 "" H 1100 9400 60  0000 C CNN
+	1    1100 9400
+	0    1    1    0
+$EndComp
+Connection ~ 1100 9400
+$Comp
+L GND #PWR?
+U 1 1 5BF87679
+P 1100 9600
+F 0 "#PWR?" H 1100 9600 30  0001 C CNN
+F 1 "GND" H 1100 9530 30  0001 C CNN
+F 2 "" H 1100 9600 60  0000 C CNN
+F 3 "" H 1100 9600 60  0000 C CNN
+	1    1100 9600
+	0    1    1    0
+$EndComp
+Connection ~ 1100 9600
 $EndSCHEMATC

Commit message: minor schematic edit and new netlist
Parts:
- gave numbers to parts that had none: 1
Changed lines of the file:
@@
 	13500 3050 14750 3050
 $Comp
-L 4081 U?
+L 4081 U17
 U 2 1 5BF8763A
 P 1700 8600
-F 0 "U?" H 1700 8650 60  0000 C CNN
+F 0 "U17" H 1700 8650 60  0000 C CNN
 F 1 "4081" H 1700 8550 60  0000 C CNN
 F 2 "" H 1700 8600 60  0000 C CNN
@@
 $EndComp
 $Comp
-L 4081 U?
+L 4081 U17
 U 3 1 5BF87645
 P 1700 9050
-F 0 "U?" H 1700 9100 60  0000 C CNN
+F 0 "U17" H 1700 9100 60  0000 C CNN
 F 1 "4081" H 1700 9000 60  0000 C CNN
 F 2 "" H 1700 9050 60  0000 C CNN
@@
 $EndComp
 $Comp
-L 4081 U?
+L 4081 U17
 U 4 1 5BF87650
 P 1700 9500
-F 0 "U?" H 1700 9550 60  0000 C CNN
+F 0 "U17" H 1700 9550 60  0000 C CNN
 F 1 "4081" H 1700 9450 60  0000 C CNN
 F 2 "" H 1700 9500 60  0000 C CNN
@@
 NoConn ~ 2300 9500
 $Comp
-L GND #PWR?
+L GND #PWR0134
 U 1 1 5BF8765B
 P 1100 8500
-F 0 "#PWR?" H 1100 8500 30  0001 C CNN
+F 0 "#PWR0134" H 1100 8500 30  0001 C CNN
 F 1 "GND" H 1100 8430 30  0001 C CNN
 F 2 "" H 1100 8500 60  0000 C CNN
@@
 Connection ~ 1100 8500
 $Comp
-L GND #PWR?
+L GND #PWR0135
 U 1 1 5BF87661
 P 1100 8700
-F 0 "#PWR?" H 1100 8700 30  0001 C CNN
+F 0 "#PWR0135" H 1100 8700 30  0001 C CNN
 F 1 "GND" H 1100 8630 30  0001 C CNN
 F 2 "" H 1100 8700 60  0000 C CNN
@@
 Connection ~ 1100 8700
 $Comp
-L GND #PWR?
+L GND #PWR0136
 U 1 1 5BF87667
 P 1100 8950
-F 0 "#PWR?" H 1100 8950 30  0001 C CNN
+F 0 "#PWR0136" H 1100 8950 30  0001 C CNN
 F 1 "GND" H 1100 8880 30  0001 C CNN
 F 2 "" H 1100 8950 60  0000 C CNN
@@
 Connection ~ 1100 8950
 $Comp
-L GND #PWR?
+L GND #PWR0137
 U 1 1 5BF8766D
 P 1100 9150
-F 0 "#PWR?" H 1100 9150 30  0001 C CNN
+F 0 "#PWR0137" H 1100 9150 30  0001 C CNN
 F 1 "GND" H 1100 9080 30  0001 C CNN
 F 2 "" H 1100 9150 60  0000 C CNN
@@
 Connection ~ 1100 9150
 $Comp
-L GND #PWR?
+L GND #PWR0138
 U 1 1 5BF87673
 P 1100 9400
-F 0 "#PWR?" H 1100 9400 30  0001 C CNN
+F 0 "#PWR0138" H 1100 9400 30  0001 C CNN
 F 1 "GND" H 1100 9330 30  0001 C CNN
 F 2 "" H 1100 9400 60  0000 C CNN
@@
 Connection ~ 1100 9400
 $Comp
-L GND #PWR?
+L GND #PWR0139
 U 1 1 5BF87679
 P 1100 9600
-F 0 "#PWR?" H 1100 9600 30  0001 C CNN
+F 0 "#PWR0139" H 1100 9600 30  0001 C CNN
 F 1 "GND" H 1100 9530 30  0001 C CNN
 F 2 "" H 1100 9600 60  0000 C CNN

Commit message: fixed unused chip connections
Parts:
- added unit 3 of U23
- added unit 4 of U23
- added unit 3 of U24
- added unit 4 of U24
- added unit 5 of U24
- added unit 6 of U24
- renumbered U4 to U24
Connections:
- no-connect marks 9 -> 15
