File: schematic/logic-clock.sch (KiCad schematic (older format))
At the start: 1 part, among them P1 AC

Commit message: started pcb
Parts:
- added P2, P3: 2-PIN_LOGIC-OUT, ~, symbol 2-PIN_LOGIC-OUT
- added P4: 4-PIN_LOGIC-OUT, ~, symbol 4-PIN_LOGIC-OUT
Connections:
- wire segments 25 -> 23
- no-connect marks 0 -> 1
Changed lines of the file:
@@
 LIBS:valves
 LIBS:kicad-custom-parts
-LIBS:logic-clock-cache
 EELAYER 27 0
 EELAYER END
@@
 L +5V #PWR03
 U 1 1 574BD962
-P 1850 3800
-F 0 "#PWR03" H 1850 3890 20  0001 C CNN
-F 1 "+5V" H 1850 3890 30  0000 C CNN
-F 2 "" H 1850 3800 60  0000 C CNN
-F 3 "" H 1850 3800 60  0000 C CNN
-	1    1850 3800
+P 1750 3800
+F 0 "#PWR03" H 1750 3890 20  0001 C CNN
+F 1 "+5V" H 1750 3890 30  0000 C CNN
+F 2 "" H 1750 3800 60  0000 C CNN
+F 3 "" H 1750 3800 60  0000 C CNN
+	1    1750 3800
 	1    0    0    -1
 $EndComp
@@
 L AC P1
 U 1 1 574BF085
-P 1650 850
-F 0 "P1" H 1400 850 50  0000 C CNN
-F 1 "AC" H 1650 950 50  0001 C CNN
-F 2 "~" H 1750 1000 60  0000 C CNN
-F 3 "~" H 1750 1000 60  0000 C CNN
-	1    1650 850
+P 1700 850
+F 0 "P1" H 1450 850 50  0000 C CNN
+F 1 "AC" H 1700 950 50  0001 C CNN
+F 2 "~" H 1800 1000 60  0000 C CNN
+F 3 "~" H 1800 1000 60  0000 C CNN
+	1    1700 850
 	0    1    1    0
 $EndComp
@@
 L +5V #PWR04
 U 1 1 574BF25F
-P 1600 1150
-F 0 "#PWR04" H 1600 1240 20  0001 C CNN
-F 1 "+5V" H 1600 1240 30  0000 C CNN
-F 2 "" H 1600 1150 60  0000 C CNN
-F 3 "" H 1600 1150 60  0000 C CNN
-	1    1600 1150
+P 1500 1150
+F 0 "#PWR04" H 1500 1240 20  0001 C CNN
+F 1 "+5V" H 1500 1240 30  0000 C CNN
+F 2 "" H 1500 1150 60  0000 C CNN
+F 3 "" H 1500 1150 60  0000 C CNN
+	1    1500 1150
 	1    0    0    -1
 $EndComp
@@
 L +5V #PWR06
 U 1 1 574BF8BC
-P 4000 750
-F 0 "#PWR06" H 4000 840 20  0001 C CNN
-F 1 "+5V" H 4000 840 30  0000 C CNN
-F 2 "" H 4000 750 60  0000 C CNN
-F 3 "" H 4000 750 60  0000 C CNN
-	1    4000 750
+P 3900 750
+F 0 "#PWR06" H 3900 840 20  0001 C CNN
+F 1 "+5V" H 3900 840 30  0000 C CNN
+F 2 "" H 3900 750 60  0000 C CNN
+F 3 "" H 3900 750 60  0000 C CNN
+	1    3900 750
 	1    0    0    -1
 $EndComp
@@
 L +5V #PWR011
 U 1 1 574C14CE
-P 1400 7300
-F 0 "#PWR011" H 1400 7390 20  0001 C CNN
-F 1 "+5V" H 1400 7390 30  0000 C CNN
-F 2 "" H 1400 7300 60  0000 C CNN
-F 3 "" H 1400 7300 60  0000 C CNN
-	1    1400 7300
+P 1600 7300
+F 0 "#PWR011" H 1600 7390 20  0001 C CNN
+F 1 "+5V" H 1600 7390 30  0000 C CNN
+F 2 "" H 1600 7300 60  0000 C CNN
+F 3 "" H 1600 7300 60  0000 C CNN
+	1    1600 7300
 	1    0    0    -1
 $EndComp
@@
 L VCC #PWR012
 U 1 1 574C1642
-P 1400 7500
-F 0 "#PWR012" H 1400 7600 30  0001 C CNN
-F 1 "VCC" H 1400 7600 30  0000 C CNN
-F 2 "" H 1400 7500 60  0000 C CNN
-F 3 "" H 1400 7500 60  0000 C CNN
-	1    1400 7500
+P 1600 7500
+F 0 "#PWR012" H 1600 7600 30  0001 C CNN
+F 1 "VCC" H 1600 7600 30  0000 C CNN
+F 2 "" H 1600 7500 60  0000 C CNN
+F 3 "" H 1600 7500 60  0000 C CNN
+	1    1600 7500
 	-1   0    0    1
 $EndComp
@@
 L VDD #PWR013
 U 1 1 574C17F3
-P 1300 7400
-F 0 "#PWR013" H 1300 7500 30  0001 C CNN
-F 1 "VDD" H 1300 7510 30  0000 C CNN
-F 2 "" H 1300 7400 60  0000 C CNN
-F 3 "" H 1300 7400 60  0000 C CNN
-	1    1300 7400
-	0    -1   -1   0
-$EndComp
-$Comp
-L PWR_FLAG #FLG014
-U 1 1 574C79C3
-P 850 7400
-F 0 "#FLG014" H 850 7495 30  0001 C CNN
-F 1 "PWR_FLAG" H 850 7580 30  0000 C CNN
-F 2 "" H 850 7400 60  0000 C CNN
-F 3 "" H 850 7400 60  0000 C CNN
-	1    850  7400
-	0    1    1    0
-$EndComp
-$Comp
-L PWR_FLAG #FLG015
-U 1 1 574C7A9E
 P 1500 7400
-F 0 "#FLG015" H 1500 7495 30  0001 C CNN
-F 1 "PWR_FLAG" H 1500 7580 30  0000 C CNN
+F 0 "#PWR013" H 1500 7500 30  0001 C CNN
+F 1 "VDD" H 1500 7510 30  0000 C CNN
 F 2 "" H 1500 7400 60  0000 C CNN
 F 3 "" H 1500 7400 60  0000 C CNN
 	1    1500 7400
+	0    -1   -1   0
+$EndComp
+$Comp
+L PWR_FLAG #FLG014
+U 1 1 574C79C3
+P 1000 7400
+F 0 "#FLG014" H 1000 7495 30  0001 C CNN
+F 1 "PWR_FLAG" H 1000 7580 30  0000 C CNN
+F 2 "" H 1000 7400 60  0000 C CNN
+F 3 "" H 1000 7400 60  0000 C CNN
+	1    1000 7400
+	0    1    1    0
+$EndComp
+$Comp
+L PWR_FLAG #FLG015
+U 1 1 574C7A9E
+P 1850 7400
+F 0 "#FLG015" H 1850 7495 30  0001 C CNN
+F 1 "PWR_FLAG" H 1850 7580 30  0000 C CNN
+F 2 "" H 1850 7400 60  0000 C CNN
+F 3 "" H 1850 7400 60  0000 C CNN
+	1    1850 7400
 	0    1    1    0
 $EndComp
@@
 	1650 3900 1700 3900
 Wire Wire Line
-	1650 3800 1850 3800
-Wire Wire Line
-	1650 3250 1700 3250
-Wire Wire Line
-	1700 3250 1700 3800
-Connection ~ 1700 3800
-Wire Wire Line
-	1650 3350 1700 3350
-Connection ~ 1700 3350
-Wire Wire Line
-	1650 3450 1700 3450
-Connection ~ 1700 3450
-Wire Wire Line
-	1650 3550 1700 3550
-Connection ~ 1700 3550
-Connection ~ 1400 800
-Connection ~ 1400 900
-Wire Wire Line
-	1400 1150 1600 1150
+	1400 1150 1500 1150
 Wire Wire Line
 	1400 1250 1450 1250
 Wire Wire Line
-	3800 750  4000 750
+	3800 750  3900 750
 Wire Wire Line
 	3800 850  3850 850
 Wire Wire Line
-	3800 950  4000 950
-Wire Wire Line
-	4000 1050 3800 1050
-Wire Wire Line
-	3800 1300 3850 1300
-Wire Wire Line
-	3850 1300 3850 1500
-Wire Wire Line
-	3850 1400 3800 1400
-Wire Wire Line
-	3850 1500 3800 1500
-Connection ~ 3850 1400
-Wire Wire Line
-	1400 1350 2600 1350
-Wire Wire Line
-	2600 1350 2600 1850
-Wire Wire Line
-	2600 1850 4000 1850
-Wire Wire Line
-	4000 1850 4000 950
-Connection ~ 4000 1050
-Wire Wire Line
-	650  7400 850  7400
+	650  7400 1000 7400
 Wire Wire Line
 	750  7300 750  7500
 Connection ~ 750  7400
 Wire Wire Line
-	1300 7400 1500 7400
-Wire Wire Line
-	1400 7300 1400 7500
-Connection ~ 1400 7400
-Wire Notes Line
-	550  7700 550  7150
-Wire Notes Line
-	550  7150 1750 7150
-Wire Notes Line
-	1750 7150 1750 7700
-Wire Notes Line
-	1750 7700 550  7700
+	1500 7400 1850 7400
+Wire Wire Line
+	1600 7300 1600 7500
+Connection ~ 1600 7400
+Wire Wire Line
+	1400 800  1450 800
+Wire Wire Line
+	1400 900  1450 900
+$Comp
+L 4-PIN_LOGIC-OUT P4
+U 1 1 574BE49F
+P 1950 3400
+F 0 "P4" H 1600 3400 50  0000 C CNN
+F 1 "4-PIN_LOGIC-OUT" H 1950 3500 50  0000 C CNN
+F 2 "~" H 2050 3550 60  0000 C CNN
+F 3 "~" H 2050 3550 60  0000 C CNN
+	1    1950 3400
+	0    1    1    0
+$EndComp
+Wire Wire Line
+	1650 3250 1700 3250
+Wire Wire Line
+	1650 3350 1700 3350
+Wire Wire Line
+	1650 3450 1700 3450
+Wire Wire Line
+	1650 3550 1700 3550
+NoConn ~ 1400 1350
+$Comp
+L +5V #PWR016
+U 1 1 574BEC1E
+P 3900 1300
+F 0 "#PWR016" H 3900 1390 20  0001 C CNN
+F 1 "+5V" H 3900 1390 30  0000 C CNN
+F 2 "" H 3900 1300 60  0000 C CNN
+F 3 "" H 3900 1300 60  0000 C CNN
+	1    3900 1300
+	1    0    0    -1
+$EndComp
+Wire Wire Line
+	3800 1300 3900 1300
+$Comp
+L 2-PIN_LOGIC-OUT P2
+U 1 1 574BEF09
+P 4200 1000
+F 0 "P2" H 3950 1000 50  0000 C CNN
+F 1 "2-PIN_LOGIC-OUT" H 4200 1100 50  0000 C CNN
+F 2 "~" H 4300 1150 60  0000 C CNN
+F 3 "~" H 4300 1150 60  0000 C CNN
+	1    4200 1000
+	0    1    1    0
+$EndComp
+Wire Wire Line
+	3800 950  3950 950
+Wire Wire Line
+	3800 1050 3950 1050
+$Comp
+L 2-PIN_LOGIC-OUT P3
+U 1 1 574BF06C
+P 4650 1450
+F 0 "P3" H 4400 1450 50  0000 C CNN
+F 1 "2-PIN_LOGIC-OUT" H 4650 1550 50  0000 C CNN
+F 2 "~" H 4750 1600 60  0000 C CNN
+F 3 "~" H 4750 1600 60  0000 C CNN
+	1    4650 1450
+	0    1    1    0
+$EndComp
+Wire Wire Line
+	3800 1400 4400 1400
+Wire Wire Line
+	3800 1500 4400 1500
+Wire Wire Line
+	1650 3800 1750 3800
+Text GLabel 900  7300 1    60   UnSpc ~ 0
+GND
+Wire Wire Line
+	900  7300 900  7400
+Connection ~ 900  7400
+Text GLabel 1750 7300 1    60   UnSpc ~ 0
++5V
+Wire Wire Line
+	1750 7300 1750 7400
+Connection ~ 1750 7400
+Wire Bus Line
+	550  7700 550  6950
+Wire Bus Line
+	550  6950 2100 6950
+Wire Bus Line
+	2100 6950 2100 7700
+Wire Bus Line
+	2100 7700 550  7700
 $EndSCHEMATC

Commit message: pcb rev 1
Parts:
- added P10, P11, P7, P8, P9: 4-PIN_LOGIC-OUT, ~, symbol 4-PIN_LOGIC-OUT
- added P12: 2-PIN_LOGIC-OUT, ~, symbol 2-PIN_LOGIC-OUT
- added R32: 0, ~, symbol USR
Connections:
- wire segments 23 -> 21

Commit message: working on schematic...
Changed lines of the file:
@@
 $Descr USLetter 11000 8500
 encoding utf-8
-Sheet 1 4
+Sheet 1 5
 Title "4000 SERIES LOGIC CLOCK w/ ALARM & RS-232 SET"
-Date "20 jun 2016"
+Date "15 jul 2016"
 Rev "1"
 Comp "Michael Craft"
@@
 	6300 6050 6350 6050
 NoConn ~ 6850 6050
+$Sheet
+S 5250 2500 3350 1750
+U 577F24F6
+F0 "logic-board" 50
+F1 "logic-board.sch" 50
+$EndSheet
 $EndSCHEMATC

Commit message: added display pwm board
Parts:
- removed P10, P11, P4, P7, P8, P9: 4-PIN_LOGIC-OUT, ~, symbol 4-PIN_LOGIC-OUT
- removed P12: 2-PIN_LOGIC-OUT, ~, symbol 2-PIN_LOGIC-OUT
- removed R32: 0, ~, symbol USR
Connections:
- wire segments 21 -> 48
- no-connect marks 1 -> 0
