File: schematic/logic-clock.sch (KiCad schematic (older format))
At the start: 3 parts, among them P1 AC, P2 2-PIN_LOGIC-OUT, P3 2-PIN_LOGIC-OUT

Commit message: schematic is "done"
Parts:
- removed P2, P3: 2-PIN_LOGIC-OUT, ~, symbol 2-PIN_LOGIC-OUT
- added P?: 3-PIN_HEADER, ~, symbol 3-PIN_HEADER
- added SW? (x2): MOMENTARY_NO, ~, symbol MOMENTARY_NO
Connections:
- net labels added: 1Hz
- wire segments 48 -> 81
Other:
- note added: "KICAD POWER NET VIRTUAL CONNECTIONS"
- note added: "NOTE: PHYSICAL BOARD WILL HAVE PASS-THRU HEADERS"
- note added: "NOTE: PHYSICAL HEADERS FOR DIGITS ARE IN ORDER ABCD"
- note added: "TO RS232 LEVEL-SHIFTER"

Commit message: added fast set
Parts:
- added SW? (x2): SWITCH_INV, ~, symbol SWITCH_INV
Connections:
- wire segments 81 -> 93
Other:
- note added: "FAST SET"
Changed lines of the file:
@@
 F33 "SET" I T 6000 2200 60
 F34 "1Hz" O B 8500 3950 60
+F35 "1Hz_OUT" O T 7100 2200 60
+F36 "10Hz_OUT" O T 7300 2200 60
+F37 "SEC_CLOCK" I T 7200 2200 60
+F38 "TEN-MIN_CLOCK" I T 6800 2200 60
+F39 "MIN-CARRY" O T 6700 2200 60
+F40 "10Hz_OUT2" O T 6900 2200 60
 $EndSheet
 $Sheet
@@
 Text Notes 5750 3650 0    60   ~ 0
 NOTE: PHYSICAL HEADERS FOR DIGITS ARE IN ORDER ABCD
-Wire Wire Line
-	1550 4000 1650 4000
-Wire Wire Line
-	1550 4100 1600 4100
-Wire Wire Line
-	650  7650 1000 7650
-Wire Wire Line
-	750  7550 750  7750
-Connection ~ 750  7650
-Wire Wire Line
-	1500 7650 1850 7650
-Wire Wire Line
-	1600 7550 1600 7750
-Connection ~ 1600 7650
-Wire Wire Line
-	900  7550 900  7650
-Connection ~ 900  7650
-Wire Wire Line
-	1750 7550 1750 7650
-Connection ~ 1750 7650
-Wire Wire Line
-	8350 6250 8350 3950
-Wire Wire Line
-	8250 6250 8250 3950
-Wire Wire Line
-	8150 6250 8150 3950
-Wire Wire Line
-	8050 6250 8050 3950
-Wire Wire Line
-	7900 6250 7900 3950
-Wire Wire Line
-	7800 6250 7800 3950
-Wire Wire Line
-	7700 6250 7700 3950
-Wire Wire Line
-	7600 6250 7600 3950
-Wire Wire Line
-	7450 6250 7450 3950
-Wire Wire Line
-	7350 6250 7350 3950
-Wire Wire Line
-	7250 6250 7250 3950
-Wire Wire Line
-	7150 6250 7150 3950
-Wire Wire Line
-	7000 6250 7000 3950
-Wire Wire Line
-	6900 6250 6900 3950
-Wire Wire Line
-	6800 6250 6800 3950
-Wire Wire Line
-	6700 6250 6700 3950
-Wire Wire Line
-	6550 6250 6550 3950
-Wire Wire Line
-	6450 6250 6450 3950
-Wire Wire Line
-	6350 6250 6350 3950
-Wire Wire Line
-	6250 6250 6250 3950
-Wire Wire Line
-	6100 6250 6100 3950
-Wire Wire Line
-	6000 6250 6000 3950
-Wire Wire Line
-	5900 6250 5900 3950
-Wire Wire Line
-	5800 6250 5800 3950
-Wire Wire Line
-	5650 6250 5650 3950
-Wire Wire Line
-	5550 6250 5550 3950
-Wire Wire Line
-	5200 1800 5200 1850
-Wire Wire Line
-	5300 1800 5300 1850
-Wire Wire Line
-	5400 1800 5400 2200
-Wire Wire Line
-	5200 2150 5200 2200
-Wire Wire Line
-	5300 2150 5300 2200
-Wire Wire Line
-	5200 1000 5200 1050
-Wire Wire Line
-	5300 1000 5300 1050
 $Comp
 L +5V #PWR?
@@
 	0    1    -1   0
 $EndComp
-Wire Wire Line
-	10300 5700 10350 5700
 $Comp
 L USGND #PWR?
@@
 	0    -1   -1   0
 $EndComp
-Wire Wire Line
-	10300 5800 10350 5800
 Text Notes 500  7250 0    60   ~ 0
 KICAD POWER NET VIRTUAL CONNECTIONS
@@
 F18 "ALARM" O L 3250 4300 60
 $EndSheet
-Wire Wire Line
-	8950 5700 8500 5700
-Wire Wire Line
-	8500 5700 8500 6250
-Wire Wire Line
-	8950 5800 8600 5800
-Wire Wire Line
-	8600 5800 8600 6250
 Text Notes 3850 6600 1    60   ~ 0
 NOTE: PHYSICAL BOARD WILL HAVE PASS-THRU HEADERS
-Wire Wire Line
-	4500 4050 7000 4050
-Connection ~ 7000 4050
-Wire Wire Line
-	4500 4150 6900 4150
-Connection ~ 6900 4150
-Wire Wire Line
-	4500 4250 6800 4250
-Connection ~ 6800 4250
-Wire Wire Line
-	4500 4350 6700 4350
-Connection ~ 6700 4350
-Wire Wire Line
-	4500 4500 6550 4500
-Connection ~ 6550 4500
-Wire Wire Line
-	4500 4600 6450 4600
-Connection ~ 6450 4600
-Wire Wire Line
-	4500 4700 6350 4700
-Connection ~ 6350 4700
-Wire Wire Line
-	4500 4800 6250 4800
-Connection ~ 6250 4800
-Wire Wire Line
-	4500 4950 6100 4950
-Connection ~ 6100 4950
-Wire Wire Line
-	4500 5050 6000 5050
-Connection ~ 6000 5050
-Wire Wire Line
-	4500 5150 5900 5150
-Connection ~ 5900 5150
-Wire Wire Line
-	4500 5250 5800 5250
-Connection ~ 5800 5250
-Wire Wire Line
-	4500 5400 5650 5400
-Connection ~ 5650 5400
-Wire Wire Line
-	4500 5500 5550 5500
-Connection ~ 5550 5500
 $Comp
 L +5V #PWR?
@@
 	0    1    1    0
 $EndComp
-Wire Wire Line
-	3200 4050 3250 4050
-Wire Wire Line
-	3200 4150 3250 4150
 $Sheet
 S 5700 1050 650  1100
@@
 Text GLabel 1800 4200 2    60   Input ~ 0
 1Hz
-Wire Wire Line
-	1550 4200 1800 4200
 Text GLabel 8500 4000 3    60   Output ~ 0
 1Hz
-Wire Wire Line
-	8500 3950 8500 4000
-Wire Wire Line
-	1550 4300 3250 4300
 $Comp
 L MOMENTARY_NO SW?
@@
 	1    0    0    -1
 $EndComp
-Wire Wire Line
-	1550 4550 1650 4550
-Wire Wire Line
-	1650 4550 1650 4400
-Wire Wire Line
-	1650 4400 2950 4400
-Wire Wire Line
-	2200 4400 2200 4650
-Wire Wire Line
-	1600 4650 1550 4650
-Wire Wire Line
-	2350 4750 1550 4750
-Wire Wire Line
-	2950 4400 2950 4750
-Connection ~ 2200 4400
-Wire Wire Line
-	5800 2150 5800 2200
-Wire Wire Line
-	5900 2150 5900 2200
-Wire Wire Line
-	6000 2150 6000 2200
 $Comp
 L +5V #PWR?
@@
 	1    0    0    1
 $EndComp
-Wire Wire Line
-	5800 1000 5800 1050
-Wire Wire Line
-	5900 1000 5900 1050
 $Comp
 L 3-PIN_HEADER P?
@@
 	1    0    0    -1
 $EndComp
-Wire Wire Line
-	6050 900  6050 1050
-Wire Wire Line
-	6150 900  6150 1050
-Wire Wire Line
-	6250 900  6250 1050
 Text Notes 6300 900  0    60   ~ 0
 TO RS232 LEVEL-SHIFTER
+Wire Wire Line
+	1550 4000 1650 4000
+Wire Wire Line
+	1550 4100 1600 4100
+Wire Wire Line
+	650  7650 1000 7650
+Wire Wire Line
+	750  7550 750  7750
+Connection ~ 750  7650
+Wire Wire Line
+	1500 7650 1850 7650
+Wire Wire Line
+	1600 7550 1600 7750
+Connection ~ 1600 7650
+Wire Wire Line
+	900  7550 900  7650
+Connection ~ 900  7650
+Wire Wire Line
+	1750 7550 1750 7650
+Connection ~ 1750 7650
+Wire Wire Line
+	8350 6250 8350 3950
+Wire Wire Line
+	8250 6250 8250 3950
+Wire Wire Line
+	8150 6250 8150 3950
+Wire Wire Line
+	8050 6250 8050 3950
+Wire Wire Line
+	7900 6250 7900 3950
+Wire Wire Line
+	7800 6250 7800 3950
+Wire Wire Line
+	7700 6250 7700 3950
+Wire Wire Line
+	7600 6250 7600 3950
+Wire Wire Line
+	7450 6250 7450 3950
+Wire Wire Line
+	7350 6250 7350 3950
+Wire Wire Line
+	7250 6250 7250 3950
+Wire Wire Line
+	7150 6250 7150 3950
+Wire Wire Line
+	7000 6250 7000 3950
+Wire Wire Line
+	6900 6250 6900 3950
+Wire Wire Line
+	6800 6250 6800 3950
+Wire Wire Line
+	6700 6250 6700 3950
+Wire Wire Line
+	6550 6250 6550 3950
+Wire Wire Line
+	6450 6250 6450 3950
+Wire Wire Line
+	6350 6250 6350 3950
+Wire Wire Line
+	6250 6250 6250 3950
+Wire Wire Line
+	6100 6250 6100 3950
+Wire Wire Line
+	6000 6250 6000 3950
+Wire Wire Line
+	5900 6250 5900 3950
+Wire Wire Line
+	5800 6250 5800 3950
+Wire Wire Line
+	5650 6250 5650 3950
+Wire Wire Line
+	5550 6250 5550 3950
+Wire Wire Line
+	5200 1800 5200 1850
+Wire Wire Line
+	5300 1800 5300 1850
+Wire Wire Line
+	5400 1800 5400 2200
+Wire Wire Line
+	5200 2150 5200 2200
+Wire Wire Line
+	5300 2150 5300 2200
+Wire Wire Line
+	5200 1000 5200 1050
+Wire Wire Line
+	5300 1000 5300 1050
+Wire Wire Line
+	10300 5700 10350 5700
+Wire Wire Line
+	10300 5800 10350 5800
+Wire Wire Line
+	8950 5700 8500 5700
+Wire Wire Line
+	8500 5700 8500 6250
+Wire Wire Line
+	8950 5800 8600 5800
+Wire Wire Line
+	8600 5800 8600 6250
+Wire Wire Line
+	4500 4050 7000 4050
+Connection ~ 7000 4050
+Wire Wire Line
+	4500 4150 6900 4150
+Connection ~ 6900 4150
+Wire Wire Line
+	4500 4250 6800 4250
+Connection ~ 6800 4250
+Wire Wire Line
+	4500 4350 6700 4350
+Connection ~ 6700 4350
+Wire Wire Line
+	4500 4500 6550 4500
+Connection ~ 6550 4500
+Wire Wire Line
+	4500 4600 6450 4600
+Connection ~ 6450 4600
+Wire Wire Line
+	4500 4700 6350 4700
+Connection ~ 6350 4700
+Wire Wire Line
+	4500 4800 6250 4800
+Connection ~ 6250 4800
+Wire Wire Line
+	4500 4950 6100 4950
+Connection ~ 6100 4950
+Wire Wire Line
+	4500 5050 6000 5050
+Connection ~ 6000 5050
+Wire Wire Line
+	4500 5150 5900 5150
+Connection ~ 5900 5150
+Wire Wire Line
+	4500 5250 5800 5250
+Connection ~ 5800 5250
+Wire Wire Line
+	4500 5400 5650 5400
+Connection ~ 5650 5400
+Wire Wire Line
+	4500 5500 5550 5500
+Connection ~ 5550 5500
+Wire Wire Line
+	3200 4050 3250 4050
+Wire Wire Line
+	3200 4150 3250 4150
+Wire Wire Line
+	1550 4200 1800 4200
+Wire Wire Line
+	8500 3950 8500 4000
+Wire Wire Line
+	1550 4300 3250 4300
+Wire Wire Line
+	1550 4550 1650 4550
+Wire Wire Line
+	1650 4550 1650 4400
+Wire Wire Line
+	1650 4400 2950 4400
+Wire Wire Line
+	2200 4400 2200 4650
+Wire Wire Line
+	1600 4650 1550 4650
+Wire Wire Line
+	2350 4750 1550 4750
+Wire Wire Line
+	2950 4400 2950 4750
+Connection ~ 2200 4400
+Wire Wire Line
+	5800 2150 5800 2200
+Wire Wire Line
+	5900 2150 5900 2200
+Wire Wire Line
+	6000 2150 6000 2200
+Wire Wire Line
+	5800 1000 5800 1050
+Wire Wire Line
+	5900 1000 5900 1050
+Wire Wire Line
+	6050 900  6050 1050
+Wire Wire Line
+	6150 900  6150 1050
+Wire Wire Line
+	6250 900  6250 1050
+Wire Wire Line
+	6700 1150 6900 1150
+Wire Wire Line
+	6800 1500 7900 1500
+Wire Wire Line
+	7900 1500 7900 1250
+Wire Wire Line
+	6700 1150 6700 2200
+Wire Wire Line
+	6800 1500 6800 2200
+Wire Wire Line
+	6900 1350 6900 2200
+Wire Wire Line
+	7300 1850 7300 2200
+Wire Wire Line
+	7100 2200 7100 1650
+Wire Wire Line
+	7100 1650 7300 1650
+Wire Wire Line
+	7200 2200 7200 2000
+Wire Wire Line
+	7200 2000 8300 2000
+Wire Wire Line
+	8300 2000 8300 1750
+Text Notes 8000 1450 0    60   ~ 0
+FAST SET
+$Comp
+L SWITCH_INV SW?
+U 1 1 57C49464
+P 7800 1750
+F 0 "SW?" H 7600 1900 50  0000 C CNN
+F 1 "SWITCH_INV" H 7650 1600 50  0000 C CNN
+F 2 "~" H 7800 1750 60  0000 C CNN
+F 3 "~" H 7800 1750 60  0000 C CNN
+	1    7800 1750
+	-1   0    0    -1
+$EndComp
+$Comp
+L SWITCH_INV SW?
+U 1 1 57C48EEE
+P 7400 1250
+F 0 "SW?" H 7200 1400 50  0000 C CNN
+F 1 "SWITCH_INV" H 7250 1100 50  0000 C CNN
+F 2 "~" H 7400 1250 60  0000 C CNN
+F 3 "~" H 7400 1250 60  0000 C CNN
+	1    7400 1250
+	-1   0    0    -1
+$EndComp
 $EndSCHEMATC
