File: schematic/logic-clock.sch (KiCad schematic (older format))
At the start: 6 parts, among them P1 AC

Commit message: passes ERC
Parts:
- gave numbers to parts that had none: 5
- renumbered P1 to P2
Changed lines of the file:
@@
 $EndSheet
 $Comp
-L AC P1
+L AC P2
 U 1 1 574BF085
 P 5250 750
-F 0 "P1" H 5000 750 50  0000 C CNN
+F 0 "P2" H 5000 750 50  0000 C CNN
 F 1 "AC" H 5250 850 50  0001 C CNN
 F 2 "~" H 5350 900 60  0000 C CNN
@@
 $EndComp
 $Comp
-L +5V #PWR02
+L +5V #PWR01
 U 1 1 574BF25F
 P 5200 1850
-F 0 "#PWR02" H 5200 1940 20  0001 C CNN
+F 0 "#PWR01" H 5200 1940 20  0001 C CNN
 F 1 "+5V" H 5200 1940 30  0000 C CNN
 F 2 "" H 5200 1850 60  0000 C CNN
@@
 $EndComp
 $Comp
-L USGND #PWR03
+L USGND #PWR02
 U 1 1 574BF3F7
 P 5300 1850
-F 0 "#PWR03" H 5300 1850 30  0001 C CNN
+F 0 "#PWR02" H 5300 1850 30  0001 C CNN
 F 1 "USGND" H 5300 1780 30  0001 C CNN
 F 2 "~" H 5300 1850 60  0000 C CNN
@@
 $EndComp
 $Comp
-L +5V #PWR04
+L +5V #PWR03
 U 1 1 574BF8BC
 P 1650 4000
-F 0 "#PWR04" H 1650 4090 20  0001 C CNN
+F 0 "#PWR03" H 1650 4090 20  0001 C CNN
 F 1 "+5V" H 1650 4090 30  0000 C CNN
 F 2 "" H 1650 4000 60  0000 C CNN
@@
 $EndComp
 $Comp
-L USGND #PWR05
+L USGND #PWR04
 U 1 1 574BFA46
 P 1600 4100
-F 0 "#PWR05" H 1600 4100 30  0001 C CNN
+F 0 "#PWR04" H 1600 4100 30  0001 C CNN
 F 1 "USGND" H 1600 4030 30  0001 C CNN
 F 2 "~" H 1600 4100 60  0000 C CNN
@@
 $EndComp
 $Comp
-L GND #PWR06
+L GND #PWR05
 U 1 1 574C0A8F
 P 650 7650
-F 0 "#PWR06" H 650 7650 30  0001 C CNN
+F 0 "#PWR05" H 650 7650 30  0001 C CNN
 F 1 "GND" H 650 7580 30  0001 C CNN
 F 2 "" H 650 7650 60  0000 C CNN
@@
 $EndComp
 $Comp
-L USGND #PWR07
+L USGND #PWR06
 U 1 1 574C0C36
 P 750 7750
-F 0 "#PWR07" H 750 7750 30  0001 C CNN
+F 0 "#PWR06" H 750 7750 30  0001 C CNN
 F 1 "USGND" H 750 7680 30  0001 C CNN
 F 2 "~" H 750 7750 60  0000 C CNN
@@
 $EndComp
 $Comp
-L VSS #PWR08
+L VSS #PWR07
 U 1 1 574C0FEA
 P 750 7550
-F 0 "#PWR08" H 750 7550 30  0001 C CNN
+F 0 "#PWR07" H 750 7550 30  0001 C CNN
 F 1 "VSS" H 750 7480 30  0000 C CNN
 F 2 "" H 750 7550 60  0000 C CNN
@@
 $EndComp
 $Comp
-L +5V #PWR09
+L +5V #PWR08
 U 1 1 574C14CE
 P 1600 7550
-F 0 "#PWR09" H 1600 7640 20  0001 C CNN
+F 0 "#PWR08" H 1600 7640 20  0001 C CNN
 F 1 "+5V" H 1600 7640 30  0000 C CNN
 F 2 "" H 1600 7550 60  0000 C CNN
@@
 $EndComp
 $Comp
-L VCC #PWR010
+L VCC #PWR09
 U 1 1 574C1642
 P 1600 7750
-F 0 "#PWR010" H 1600 7850 30  0001 C CNN
+F 0 "#PWR09" H 1600 7850 30  0001 C CNN
 F 1 "VCC" H 1600 7850 30  0000 C CNN
 F 2 "" H 1600 7750 60  0000 C CNN
@@
 $EndComp
 $Comp
-L VDD #PWR011
+L VDD #PWR010
 U 1 1 574C17F3
 P 1500 7650
-F 0 "#PWR011" H 1500 7750 30  0001 C CNN
+F 0 "#PWR010" H 1500 7750 30  0001 C CNN
 F 1 "VDD" H 1500 7760 30  0000 C CNN
 F 2 "" H 1500 7650 60  0000 C CNN
@@
 $EndComp
 $Comp
-L PWR_FLAG #FLG012
+L PWR_FLAG #FLG011
 U 1 1 574C79C3
 P 1000 7650
-F 0 "#FLG012" H 1000 7745 30  0001 C CNN
+F 0 "#FLG011" H 1000 7745 30  0001 C CNN
 F 1 "PWR_FLAG" H 1000 7830 30  0000 C CNN
 F 2 "" H 1000 7650 60  0000 C CNN
@@
 $EndComp
 $Comp
-L PWR_FLAG #FLG013
+L PWR_FLAG #FLG012
 U 1 1 574C7A9E
 P 1850 7650
-F 0 "#FLG013" H 1850 7745 30  0001 C CNN
+F 0 "#FLG012" H 1850 7745 30  0001 C CNN
 F 1 "PWR_FLAG" H 1850 7830 30  0000 C CNN
 F 2 "" H 1850 7650 60  0000 C CNN
@@
 +5V
 $Comp
-L +5V #PWR?
+L +5V #PWR013
 U 1 1 57C0527A
 P 5200 2150
-F 0 "#PWR?" H 5200 2240 20  0001 C CNN
+F 0 "#PWR013" H 5200 2240 20  0001 C CNN
 F 1 "+5V" H 5200 2240 30  0000 C CNN
 F 2 "" H 5200 2150 60  0000 C CNN
@@
 $EndComp
 $Comp
-L USGND #PWR?
+L USGND #PWR014
 U 1 1 57C05718
 P 5300 2150
-F 0 "#PWR?" H 5300 2150 30  0001 C CNN
+F 0 "#PWR014" H 5300 2150 30  0001 C CNN
 F 1 "USGND" H 5300 2080 30  0001 C CNN
 F 2 "~" H 5300 2150 60  0000 C CNN
@@
 NOTE: PHYSICAL HEADERS FOR DIGITS ARE IN ORDER ABCD
 $Comp
-L +5V #PWR?
+L +5V #PWR015
 U 1 1 57C39E1A
 P 10350 5700
-F 0 "#PWR?" H 10350 5790 20  0001 C CNN
+F 0 "#PWR015" H 10350 5790 20  0001 C CNN
 F 1 "+5V" H 10350 5790 30  0000 C CNN
 F 2 "" H 10350 5700 60  0000 C CNN
@@
 $EndComp
 $Comp
-L USGND #PWR?
+L USGND #PWR016
 U 1 1 57C39FE5
 P 10350 5800
-F 0 "#PWR?" H 10350 5800 30  0001 C CNN
+F 0 "#PWR016" H 10350 5800 30  0001 C CNN
 F 1 "USGND" H 10350 5730 30  0001 C CNN
 F 2 "~" H 10350 5800 60  0000 C CNN
@@
 NOTE: PHYSICAL BOARD WILL HAVE PASS-THRU HEADERS
 $Comp
-L +5V #PWR?
+L +5V #PWR017
 U 1 1 57C42932
 P 3200 4050
-F 0 "#PWR?" H 3200 4140 20  0001 C CNN
+F 0 "#PWR017" H 3200 4140 20  0001 C CNN
 F 1 "+5V" H 3200 4140 30  0000 C CNN
 F 2 "" H 3200 4050 60  0000 C CNN
@@
 $EndComp
 $Comp
-L USGND #PWR?
+L USGND #PWR018
 U 1 1 57C42C4C
 P 3200 4150
-F 0 "#PWR?" H 3200 4150 30  0001 C CNN
+F 0 "#PWR018" H 3200 4150 30  0001 C CNN
 F 1 "USGND" H 3200 4080 30  0001 C CNN
 F 2 "~" H 3200 4150 60  0000 C CNN
@@
 1Hz
 $Comp
-L MOMENTARY_NO SW?
+L MOMENTARY_NO SW3
 U 1 1 57C3E3E0
 P 1900 4650
-F 0 "SW?" H 2025 4800 50  0000 C CNN
+F 0 "SW3" H 2025 4800 50  0000 C CNN
 F 1 "MOMENTARY_NO" H 1900 4570 50  0001 C CNN
 F 2 "~" H 1900 4650 60  0000 C CNN
@@
 $EndComp
 $Comp
-L MOMENTARY_NO SW?
+L MOMENTARY_NO SW4
 U 1 1 57C3E56B
 P 2650 4750
-F 0 "SW?" H 2775 4900 50  0000 C CNN
+F 0 "SW4" H 2775 4900 50  0000 C CNN
 F 1 "MOMENTARY_NO" H 2650 4670 50  0001 C CNN
 F 2 "~" H 2650 4750 60  0000 C CNN
@@
 $EndComp
 $Comp
-L +5V #PWR?
+L +5V #PWR019
 U 1 1 57C4038F
 P 5800 1000
-F 0 "#PWR?" H 5800 1090 20  0001 C CNN
+F 0 "#PWR019" H 5800 1090 20  0001 C CNN
 F 1 "+5V" H 5800 1090 30  0000 C CNN
 F 2 "" H 5800 1000 60  0000 C CNN
@@
 $EndComp
 $Comp
-L USGND #PWR?
+L USGND #PWR020
 U 1 1 57C40395
 P 5900 1000
-F 0 "#PWR?" H 5900 1000 30  0001 C CNN
+F 0 "#PWR020" H 5900 1000 30  0001 C CNN
 F 1 "USGND" H 5900 930 30  0001 C CNN
 F 2 "~" H 5900 1000 60  0000 C CNN
@@
 $EndComp
 $Comp
-L 3-PIN_HEADER P?
+L 3-PIN_HEADER P1
 U 1 1 57C40C08
 P 6150 650
-F 0 "P?" H 5850 650 50  0000 C CNN
+F 0 "P1" H 5850 650 50  0000 C CNN
 F 1 "3-PIN_HEADER" H 6150 850 50  0001 C CNN
 F 2 "~" H 6200 800 60  0000 C CNN
@@
 FAST SET
 $Comp
-L SWITCH_INV SW?
+L SWITCH_INV SW2
 U 1 1 57C49464
 P 7800 1750
-F 0 "SW?" H 7600 1900 50  0000 C CNN
+F 0 "SW2" H 7600 1900 50  0000 C CNN
 F 1 "SWITCH_INV" H 7650 1600 50  0000 C CNN
 F 2 "~" H 7800 1750 60  0000 C CNN
@@
 $EndComp
 $Comp
-L SWITCH_INV SW?
+L SWITCH_INV SW1
 U 1 1 57C48EEE
 P 7400 1250
-F 0 "SW?" H 7200 1400 50  0000 C CNN
+F 0 "SW1" H 7200 1400 50  0000 C CNN
 F 1 "SWITCH_INV" H 7250 1100 50  0000 C CNN
 F 2 "~" H 7400 1250 60  0000 C CNN
