File: schematic/display-pwm-board.sch (KiCad schematic (older format))
At the start: 9 parts

Commit message: schematic is "done"
Parts:
- R?: value 18K -> 1K8
Connections:
- net labels added: +5V_OUT
Changed lines of the file:
@@
 EELAYER 27 0
 EELAYER END
-$Descr A4 11693 8268
+$Descr USLetter 11000 8500
 encoding utf-8
-Sheet 6 6
-Title "DISPLAY PWM SIGNAL GENERATOR"
-Date "25 aug 2016"
+Sheet 4 8
+Title "LOGIC CLOCK DISPLAY PWM SIGNAL GENERATOR"
+Date "28 aug 2016"
 Rev "1"
 Comp "Michael Craft"
@@
 P 3700 3250
 F 0 "R?" V 3780 3250 40  0000 C CNN
-F 1 "18K" V 3600 3250 40  0000 C CNN
+F 1 "1K8" V 3600 3250 40  0000 C CNN
 F 2 "~" V 3630 3250 30  0000 C CNN
 F 3 "~" H 3700 3250 30  0000 C CNN
@@
 $EndComp
 Text HLabel 8100 2600 2    60   Output ~ 0
-+5V
++5V_OUT
 $Comp
 L +5V #PWR?

Commit message: started rs232 board
Parts:
- added D?: LED, ~, symbol LED
- added R?: 1K, ~, symbol USR
Changed lines of the file:
@@
 Sheet 4 8
 Title "LOGIC CLOCK DISPLAY PWM SIGNAL GENERATOR"
-Date "28 aug 2016"
+Date "29 aug 2016"
 Rev "1"
 Comp "Michael Craft"
@@
 Wire Notes Line
 	8100 2500 8100 2800
+$Comp
+L LED D?
+U 1 1 57C38BBE
+P 7450 2200
+F 0 "D?" H 7450 2300 50  0000 C CNN
+F 1 "LED" H 7450 2100 50  0000 C CNN
+F 2 "~" H 7450 2200 60  0000 C CNN
+F 3 "~" H 7450 2200 60  0000 C CNN
+	1    7450 2200
+	0    -1   -1   0
+$EndComp
+$Comp
+L USR R?
+U 1 1 57C38BF4
+P 7450 2650
+F 0 "R?" V 7530 2650 40  0000 C CNN
+F 1 "1K" V 7350 2650 40  0000 C CNN
+F 2 "~" V 7380 2650 30  0000 C CNN
+F 3 "~" H 7450 2650 30  0000 C CNN
+	1    7450 2650
+	1    0    0    -1
+$EndComp
+Connection ~ 7450 2900
+Connection ~ 7450 2400
+$Comp
+L USGND #PWR?
+U 1 1 57C38C13
+P 7450 2000
+F 0 "#PWR?" H 7450 2000 30  0001 C CNN
+F 1 "USGND" H 7450 1930 30  0001 C CNN
+F 2 "~" H 7450 2000 60  0000 C CNN
+F 3 "~" H 7450 2000 60  0000 C CNN
+	1    7450 2000
+	-1   0    0    1
+$EndComp
+Connection ~ 7450 2000
 $EndSCHEMATC

Commit message: passes ERC
Parts:
- gave numbers to parts that had none: 10
Changed lines of the file:
@@
 $EndDescr
 $Comp
-L 4584 U?
-U 1 1 57C38398
+L 4584 U4
+U 4 1 57C38398
 P 3700 2900
-F 0 "U?" H 3850 3000 40  0000 C CNN
+F 0 "U4" H 3850 3000 40  0000 C CNN
 F 1 "4584" H 3900 2800 40  0000 C CNN
 F 2 "~" H 3650 2900 60  0000 C CNN
 F 3 "~" H 3650 2900 60  0000 C CNN
-	1    3700 2900
-	1    0    0    -1
-$EndComp
-$Comp
-L USR R?
+	4    3700 2900
+	1    0    0    -1
+$EndComp
+$Comp
+L USR R27
 U 1 1 57C383A7
 P 3700 3250
-F 0 "R?" V 3780 3250 40  0000 C CNN
+F 0 "R27" V 3780 3250 40  0000 C CNN
 F 1 "1K8" V 3600 3250 40  0000 C CNN
 F 2 "~" V 3630 3250 30  0000 C CNN
@@
 $EndComp
 $Comp
-L C C?
+L C C15
 U 1 1 57C383CE
 P 3250 3450
-F 0 "C?" H 3250 3550 40  0000 L CNN
+F 0 "C15" H 3250 3550 40  0000 L CNN
 F 1 "100nF" H 3256 3365 40  0000 L CNN
 F 2 "~" H 3288 3300 30  0000 C CNN
@@
 $EndComp
 $Comp
-L USGND #PWR?
+L USGND #PWR078
 U 1 1 57C383EC
 P 3250 3650
-F 0 "#PWR?" H 3250 3650 30  0001 C CNN
+F 0 "#PWR078" H 3250 3650 30  0001 C CNN
 F 1 "USGND" H 3250 3580 30  0001 C CNN
 F 2 "~" H 3250 3650 60  0000 C CNN
@@
 APPROX 900Hz 80% DUTY CYCLE
 $Comp
-L 4017 U?
+L 4017 U12
 U 1 1 57C38E85
 P 5300 3450
-F 0 "U?" H 5200 3300 60  0000 C CNN
+F 0 "U12" H 5200 3300 60  0000 C CNN
 F 1 "4017" H 5200 3150 60  0000 C CNN
 F 2 "" H 5300 3450 60  0000 C CNN
@@
 $EndComp
 $Comp
-L USGND #PWR?
+L USGND #PWR079
 U 1 1 57C38E9C
 P 4650 3200
-F 0 "#PWR?" H 4650 3200 30  0001 C CNN
+F 0 "#PWR079" H 4650 3200 30  0001 C CNN
 F 1 "USGND" H 4650 3130 30  0001 C CNN
 F 2 "~" H 4650 3200 60  0000 C CNN
@@
 $EndComp
 $Comp
-L DIODE D?
+L DIODE D22
 U 1 1 57C38EC4
 P 6150 2900
-F 0 "D?" H 6150 3000 40  0000 C CNN
+F 0 "D22" H 6150 3000 40  0000 C CNN
 F 1 "DIODE" H 6150 2800 40  0001 C CNN
 F 2 "~" H 6150 2900 60  0000 C CNN
@@
 $EndComp
 $Comp
-L DIODE D?
+L DIODE D23
 U 1 1 57C38ED6
 P 6150 3000
-F 0 "D?" H 6150 3100 40  0000 C CNN
+F 0 "D23" H 6150 3100 40  0000 C CNN
 F 1 "DIODE" H 6150 2900 40  0001 C CNN
 F 2 "~" H 6150 3000 60  0000 C CNN
@@
 $EndComp
 $Comp
-L USR R?
+L USR R28
 U 1 1 57C38EDE
 P 6350 3250
-F 0 "R?" V 6430 3250 40  0000 C CNN
+F 0 "R28" V 6430 3250 40  0000 C CNN
 F 1 "100K" V 6250 3250 40  0000 C CNN
 F 2 "~" V 6280 3250 30  0000 C CNN
@@
 $EndComp
 $Comp
-L USGND #PWR?
+L USGND #PWR080
 U 1 1 57C38EEB
 P 6350 3500
-F 0 "#PWR?" H 6350 3500 30  0001 C CNN
+F 0 "#PWR080" H 6350 3500 30  0001 C CNN
 F 1 "USGND" H 6350 3430 30  0001 C CNN
 F 2 "~" H 6350 3500 60  0000 C CNN
@@
 $EndComp
 $Comp
-L 4584 U?
-U 2 1 57C38F03
+L 4584 U4
+U 5 1 57C38F03
 P 7000 2900
-F 0 "U?" H 7150 3000 40  0000 C CNN
+F 0 "U4" H 7150 3000 40  0000 C CNN
 F 1 "4584" H 7200 2800 40  0000 C CNN
 F 2 "~" H 6950 2900 60  0000 C CNN
 F 3 "~" H 6950 2900 60  0000 C CNN
-	2    7000 2900
+	5    7000 2900
 	1    0    0    -1
 $EndComp
@@
 NoConn ~ 5950 4000
 $Comp
-L USGND #PWR?
+L USGND #PWR081
 U 1 1 57C38F1D
 P 4650 3000
-F 0 "#PWR?" H 4650 3000 30  0001 C CNN
+F 0 "#PWR081" H 4650 3000 30  0001 C CNN
 F 1 "USGND" H 4650 2930 30  0001 C CNN
 F 2 "~" H 4650 3000 60  0000 C CNN
@@
 GND
 $Comp
-L MOSFET_N Q?
+L MOSFET_N Q4
 U 1 1 57C39E6A
 P 7750 2900
-F 0 "Q?" H 7760 3070 60  0000 R CNN
+F 0 "Q4" H 7760 3070 60  0000 R CNN
 F 1 "ZVN4206" H 7760 2750 60  0000 R CNN
 F 2 "~" H 7750 2900 60  0000 C CNN
@@
 $EndComp
 $Comp
-L USGND #PWR?
+L USGND #PWR082
 U 1 1 57C3A56F
 P 7850 3100
-F 0 "#PWR?" H 7850 3100 30  0001 C CNN
+F 0 "#PWR082" H 7850 3100 30  0001 C CNN
 F 1 "USGND" H 7850 3030 30  0001 C CNN
 F 2 "~" H 7850 3100 60  0000 C CNN
@@
 $EndComp
 $Comp
-L USGND #PWR?
+L USGND #PWR083
 U 1 1 57C3A5A1
 P 8050 2300
-F 0 "#PWR?" H 8050 2300 30  0001 C CNN
+F 0 "#PWR083" H 8050 2300 30  0001 C CNN
 F 1 "USGND" H 8050 2230 30  0001 C CNN
 F 2 "~" H 8050 2300 60  0000 C CNN
@@
 $EndComp
 $Comp
-L +5V #PWR?
+L +5V #PWR084
 U 1 1 57C3A5A9
 P 8050 2200
-F 0 "#PWR?" H 8050 2290 20  0001 C CNN
+F 0 "#PWR084" H 8050 2290 20  0001 C CNN
 F 1 "+5V" H 8050 2290 30  0000 C CNN
 F 2 "" H 8050 2200 60  0000 C CNN
@@
 +5V_OUT
 $Comp
-L +5V #PWR?
+L +5V #PWR085
 U 1 1 57C3A8D9
 P 8050 2600
-F 0 "#PWR?" H 8050 2690 20  0001 C CNN
+F 0 "#PWR085" H 8050 2690 20  0001 C CNN
 F 1 "+5V" H 8050 2690 30  0000 C CNN
 F 2 "" H 8050 2600 60  0000 C CNN
@@
 	8100 2500 8100 2800
 $Comp
-L LED D?
+L LED D21
 U 1 1 57C38BBE
 P 7450 2200
-F 0 "D?" H 7450 2300 50  0000 C CNN
+F 0 "D21" H 7450 2300 50  0000 C CNN
 F 1 "LED" H 7450 2100 50  0000 C CNN
 F 2 "~" H 7450 2200 60  0000 C CNN
@@
 $EndComp
 $Comp
-L USR R?
+L USR R26
 U 1 1 57C38BF4
 P 7450 2650
-F 0 "R?" V 7530 2650 40  0000 C CNN
+F 0 "R26" V 7530 2650 40  0000 C CNN
 F 1 "1K" V 7350 2650 40  0000 C CNN
 F 2 "~" V 7380 2650 30  0000 C CNN
@@
 Connection ~ 7450 2400
 $Comp
-L USGND #PWR?
+L USGND #PWR086
 U 1 1 57C38C13
 P 7450 2000
-F 0 "#PWR?" H 7450 2000 30  0001 C CNN
+F 0 "#PWR086" H 7450 2000 30  0001 C CNN
 F 1 "USGND" H 7450 1930 30  0001 C CNN
 F 2 "~" H 7450 2000 60  0000 C CNN
