File: schematic/comparator-board.sch (KiCad schematic (older format))
At the start: 0 parts

Commit message: started comparator board
Parts:
- added C?: 1uF, ~, symbol C
- added D?: DIODE, ~, symbol DIODE
- added D? (x2): LED, ~, symbol LED
- added R? (x2): 1K, ~, symbol USR
- added RR? (x2): RR8, ~, symbol RR8
- added SW? (x2): DIP-SW-8, ~, symbol DIP-SW-8
- added U? (x4): 4585, ~, symbol 4585
Connections:
- wire segments 2 -> 104
- no-connect marks 1 -> 11
Other:
- note added: "GENERATE PULSE"
- note removed: "leave space for the header parts i might need\n"

Commit message: "v1.0" Schematics are "finished". Final assembly is not yet complete and changes may be required. Everything has been tested, at least by itself.
Parts:
- added C?: 510pF, ~, symbol C
- added R?: 22K, ~, symbol USR
- added U? (x2): 4050, symbol 4050
Connections:
- wire segments 104 -> 93
- no-connect marks 11 -> 10
Other:
- moved on the sheet: C?, D?, R?
