File: schematic/rs232-board.sch (KiCad schematic (older format))
At the start: 0 parts

Commit message: started rs232 board
Parts:
- added C?: 500pF, ~, symbol C
- added C?: 1800pF, ~, symbol C
- added Q?: ZVN4206, ~, symbol MOSFET_N
- added R?: 100K, ~, symbol USR
- added R? (x2): 22K, ~, symbol USR
- added R? (x2): 82K, ~, symbol USR
- added U? (x2): 4013, symbol 4013
- added U?: 4017, symbol 4017
- added U? (x4): 4011, symbol 4011
- added U?: 4094, ~, symbol 4094
Connections:
- wire segments 4 -> 43
- no-connect marks 4 -> 13

Commit message: minutes and seconds digits confirmed working, hours needs work
Parts:
- removed C?: 500pF, ~, symbol C
- removed C?: 1800pF, ~, symbol C
- removed Q?: ZVN4206, ~, symbol MOSFET_N
- removed R?: 100K, ~, symbol USR
- removed R? (x2): 22K, ~, symbol USR
- removed R? (x2): 82K, ~, symbol USR
- removed U? (x2): 4013, symbol 4013
- removed U?: 4017, symbol 4017
- removed U? (x4): 4011, symbol 4011
- added C?: 510pF, ~, symbol C
- added C? (x2): 1800pF, ~, symbol C
- added D? (x4): DIODE, ~, symbol DIODE
- added Q?: MOSFET_P, ~, symbol MOSFET_P
- added R?: 75K, ~, symbol USR
- added R?: 22K, ~, symbol USR
- added R?: 47K 1%, ~, symbol USR
- added R?: 1K3 1%, ~, symbol USR
- added R? (x2): 10K, ~, symbol USR
- added RV?: 470R, ~, symbol POT
- added U? (x2): 4013, symbol 4013
- added U? (x4): 4584, ~, symbol 4584
- added U?: 4017, symbol 4017
Connections:
- wire segments 43 -> 41
- no-connect marks 13 -> 14
Other:
- note added: "TARGET VALUE APPROX. 48K5"

Commit message: passes ERC
Parts:
- U16: renamed from U?; symbol 4013 -> CD4013
- gave numbers to parts that had none: 19
Connections:
- no-connect marks 14 -> 22
