File: schematic/rs232-board.sch (KiCad schematic (older format))
At the start: 20 parts, among them Q7 MOSFET_P, U16 4013, U24 4584, U28 4094, U29 4017, U30 4013

Commit message: fixed unused chip connections
Parts:
- renumbered U24 to U96, U24 to U97, U24 to U98, U24 to U99
Changed lines of the file:
@@
 GND
 $Comp
-L +5V #PWR0148
+L +5V #PWR0156
 U 1 1 57C43B52
 P 1400 2700
-F 0 "#PWR0148" H 1400 2790 20  0001 C CNN
+F 0 "#PWR0156" H 1400 2790 20  0001 C CNN
 F 1 "+5V" H 1400 2790 30  0000 C CNN
 F 2 "" H 1400 2700 60  0000 C CNN
@@
 $EndComp
 $Comp
-L USGND #PWR0149
+L USGND #PWR0157
 U 1 1 57C43B61
 P 1400 2800
-F 0 "#PWR0149" H 1400 2800 30  0001 C CNN
+F 0 "#PWR0157" H 1400 2800 30  0001 C CNN
 F 1 "USGND" H 1400 2730 30  0001 C CNN
 F 2 "~" H 1400 2800 60  0000 C CNN
@@
 GND_OUT
 $Comp
-L +5V #PWR0150
+L +5V #PWR0158
 U 1 1 57C3F13A
 P 1400 3150
-F 0 "#PWR0150" H 1400 3240 20  0001 C CNN
+F 0 "#PWR0158" H 1400 3240 20  0001 C CNN
 F 1 "+5V" H 1400 3240 30  0000 C CNN
 F 2 "" H 1400 3150 60  0000 C CNN
@@
 $EndComp
 $Comp
-L USGND #PWR0151
+L USGND #PWR0159
 U 1 1 57C3F140
 P 1400 3250
-F 0 "#PWR0151" H 1400 3250 30  0001 C CNN
+F 0 "#PWR0159" H 1400 3250 30  0001 C CNN
 F 1 "USGND" H 1400 3180 30  0001 C CNN
 F 2 "~" H 1400 3250 60  0000 C CNN
@@
 $EndComp
 $Comp
-L +5V #PWR0152
+L +5V #PWR0160
 U 1 1 57C3AD70
 P 9700 2400
-F 0 "#PWR0152" H 9700 2490 20  0001 C CNN
+F 0 "#PWR0160" H 9700 2490 20  0001 C CNN
 F 1 "+5V" H 9700 2490 30  0000 C CNN
 F 2 "" H 9700 2400 60  0000 C CNN
@@
 $EndComp
 $Comp
-L USGND #PWR0153
+L USGND #PWR0161
 U 1 1 57C3AD76
 P 9700 2500
-F 0 "#PWR0153" H 9700 2500 30  0001 C CNN
+F 0 "#PWR0161" H 9700 2500 30  0001 C CNN
 F 1 "USGND" H 9700 2430 30  0001 C CNN
 F 2 "~" H 9700 2500 60  0000 C CNN
@@
 NoConn ~ 9700 2100
 $Comp
-L +5V #PWR0154
+L +5V #PWR0162
 U 1 1 57C3AF02
 P 8200 2500
-F 0 "#PWR0154" H 8200 2590 20  0001 C CNN
+F 0 "#PWR0162" H 8200 2590 20  0001 C CNN
 F 1 "+5V" H 8200 2590 30  0000 C CNN
 F 2 "" H 8200 2500 60  0000 C CNN
@@
 $EndComp
 $Comp
-L 4584 U24
+L 4584 U99
 U 2 1 582279EF
 P 2000 3350
-F 0 "U24" H 2150 3450 40  0000 C CNN
+F 0 "U99" H 2150 3450 40  0000 C CNN
 F 1 "4584" H 2200 3250 40  0000 C CNN
 F 2 "~" H 1950 3350 60  0000 C CNN
@@
 $EndComp
 $Comp
-L USGND #PWR0155
+L USGND #PWR0163
 U 1 1 58227C19
 P 2900 3900
-F 0 "#PWR0155" H 2900 3900 30  0001 C CNN
+F 0 "#PWR0163" H 2900 3900 30  0001 C CNN
 F 1 "USGND" H 2900 3830 30  0001 C CNN
 F 2 "~" H 2900 3900 60  0000 C CNN
@@
 $EndComp
 $Comp
-L USGND #PWR0156
+L USGND #PWR0164
 U 1 1 58227C1F
 P 3400 3700
-F 0 "#PWR0156" H 3400 3700 30  0001 C CNN
+F 0 "#PWR0164" H 3400 3700 30  0001 C CNN
 F 1 "USGND" H 3400 3630 30  0001 C CNN
 F 2 "~" H 3400 3700 60  0000 C CNN
@@
 $EndComp
 $Comp
-L USGND #PWR0157
+L USGND #PWR0165
 U 1 1 58227C25
 P 3400 3900
-F 0 "#PWR0157" H 3400 3900 30  0001 C CNN
+F 0 "#PWR0165" H 3400 3900 30  0001 C CNN
 F 1 "USGND" H 3400 3830 30  0001 C CNN
 F 2 "~" H 3400 3900 60  0000 C CNN
@@
 NoConn ~ 4600 4100
 $Comp
-L 4584 U24
+L 4584 U98
 U 3 1 58227C30
 P 6300 3500
-F 0 "U24" H 6450 3600 40  0000 C CNN
+F 0 "U98" H 6450 3600 40  0000 C CNN
 F 1 "4584" H 6500 3400 40  0000 C CNN
 F 2 "~" H 6250 3500 60  0000 C CNN
@@
 $EndComp
 $Comp
-L USGND #PWR0158
+L USGND #PWR0166
 U 1 1 582282BC
 P 5850 3950
-F 0 "#PWR0158" H 5850 3950 30  0001 C CNN
+F 0 "#PWR0166" H 5850 3950 30  0001 C CNN
 F 1 "USGND" H 5850 3880 30  0001 C CNN
 F 2 "~" H 5850 3950 60  0000 C CNN
@@
 $EndComp
 $Comp
-L USGND #PWR0159
+L USGND #PWR0167
 U 1 1 58229D61
 P 5500 3950
-F 0 "#PWR0159" H 5500 3950 30  0001 C CNN
+F 0 "#PWR0167" H 5500 3950 30  0001 C CNN
 F 1 "USGND" H 5500 3880 30  0001 C CNN
 F 2 "~" H 5500 3950 60  0000 C CNN
@@
 $EndComp
 $Comp
-L +5V #PWR0160
+L +5V #PWR0168
 U 1 1 58239185
 P 5200 3900
-F 0 "#PWR0160" H 5200 3990 20  0001 C CNN
+F 0 "#PWR0168" H 5200 3990 20  0001 C CNN
 F 1 "+5V" H 5200 3990 30  0000 C CNN
 F 2 "" H 5200 3900 60  0000 C CNN
@@
 $EndComp
 $Comp
-L +5V #PWR0161
+L +5V #PWR0169
 U 1 1 5823AE99
 P 7100 3600
-F 0 "#PWR0161" H 7100 3690 20  0001 C CNN
+F 0 "#PWR0169" H 7100 3690 20  0001 C CNN
 F 1 "+5V" H 7100 3690 30  0000 C CNN
 F 2 "" H 7100 3600 60  0000 C CNN
@@
 	9700 2200 10050 2200
 $Comp
-L 4584 U24
+L 4584 U97
 U 5 1 582523D9
 P 10200 4700
-F 0 "U24" H 10350 4800 40  0000 C CNN
+F 0 "U97" H 10350 4800 40  0000 C CNN
 F 1 "4584" H 10400 4600 40  0000 C CNN
 F 2 "~" H 10150 4700 60  0000 C CNN
@@
 Connection ~ 8500 4300
 $Comp
-L USGND #PWR0162
+L USGND #PWR0170
 U 1 1 58252520
 P 8200 5150
-F 0 "#PWR0162" H 8200 5150 30  0001 C CNN
+F 0 "#PWR0170" H 8200 5150 30  0001 C CNN
 F 1 "USGND" H 8200 5080 30  0001 C CNN
 F 2 "~" H 8200 5150 60  0000 C CNN
@@
 Connection ~ 8200 5150
 $Comp
-L USGND #PWR0163
+L USGND #PWR0171
 U 1 1 58252526
 P 8200 5350
-F 0 "#PWR0163" H 8200 5350 30  0001 C CNN
+F 0 "#PWR0171" H 8200 5350 30  0001 C CNN
 F 1 "USGND" H 8200 5280 30  0001 C CNN
 F 2 "~" H 8200 5350 60  0000 C CNN
@@
 $EndComp
 $Comp
-L +5V #PWR0164
+L +5V #PWR0172
 U 1 1 5825257D
 P 9800 4650
-F 0 "#PWR0164" H 9800 4740 20  0001 C CNN
+F 0 "#PWR0172" H 9800 4740 20  0001 C CNN
 F 1 "+5V" H 9800 4740 30  0000 C CNN
 F 2 "" H 9800 4650 60  0000 C CNN
@@
 Connection ~ 9800 4650
 $Comp
-L 4584 U24
+L 4584 U96
 U 4 1 58252588
 P 6750 3950
-F 0 "U24" H 6900 4050 40  0000 C CNN
+F 0 "U96" H 6900 4050 40  0000 C CNN
 F 1 "4584" H 6950 3850 40  0000 C CNN
 F 2 "~" H 6700 3950 60  0000 C CNN
@@
 	10200 3850 10400 3850
 $Comp
-L +5V #PWR0165
+L +5V #PWR0173
 U 1 1 582527ED
 P 10400 3350
-F 0 "#PWR0165" H 10400 3440 20  0001 C CNN
+F 0 "#PWR0173" H 10400 3440 20  0001 C CNN
 F 1 "+5V" H 10400 3440 30  0000 C CNN
 F 2 "" H 10400 3350 60  0000 C CNN

Commit message: half laid out, fixed netlist again
Parts:
- renumbered U16 to U89
Changed lines of the file:
@@
 Sheet 8 8
 Title "LOGIC CLOCK RS232 RECEIVER BOARD"
-Date "23 nov 2018"
+Date "24 nov 2018"
 Rev "1"
 Comp "Michael Craft"
@@
 $EndComp
 $Comp
-L CD4013 U16
+L CD4013 U89
 U 2 1 582279E2
 P 4000 3900
-F 0 "U16" H 4150 4200 60  0000 C CNN
+F 0 "U89" H 4150 4200 60  0000 C CNN
 F 1 "4013" H 4050 3600 60  0000 L CNN
 F 2 "" H 4000 3900 60  0000 C CNN

Commit message: working on RS232 receiver
Parts:
- added C?: 10pF, ~, symbol CSMALL
- added unit 5 of U99
- added unit 6 of U99
- renumbered U30 to U89, U98 to U99, U97 to U99, U96 to U99
Connections:
- wire segments 41 -> 43
- no-connect marks 22 -> 21
Other:
- note added: "BYTE OVER, RESET"
- note added: "CLOCK"
- note added: "CLOCK RECOVERY"
- note added: "DATA"
- note added: "DETECT SECRET WORD"
- note added: "OSCILLATOR TUNED FOR 9600 BAUD (9K6 HZ)"
- note added: "TARGET VALUE APPROX. 48K7"
- note removed: "TARGET VALUE APPROX. 48K5"
- moved on the sheet: C34, C35, C36, D45, D46, D47, D48, R42, R43, R44, R45, R46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

Commit message: still working on rs232
Connections:
- wire segments 43 -> 47
Other:
- moved on the sheet: C34, C35, C36, D45, D46, D47, D48, R42, R43, R44, R45, R46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

Commit message: RS232 should be done now, still untested
Parts:
- added D? (x2): DIODE, ~, symbol DIODE
- added R?: 100K, ~, symbol USR
- added U?: 4585, ~, symbol 4585
Connections:
- wire segments 47 -> 66
- no-connect marks 21 -> 19
Changed lines of the file:
@@
 Sheet 8 8
 Title "LOGIC CLOCK RS232 RECEIVER BOARD"
-Date "27 nov 2018"
-Rev "1"
+Date "28 nov 2018"
+Rev "2"
 Comp "Michael Craft"
 Comment1 ""
@@
 Connection ~ 9500 1400
 Wire Wire Line
-	2650 4500 2750 4500
+	2650 4500 2700 4500
+Wire Wire Line
+	2700 4500 2750 4500
 Wire Wire Line
 	3250 4500 3800 4500
@@
 Connection ~ 5800 4300
 Wire Wire Line
-	5000 4650 5650 4650
-Wire Wire Line
-	5300 4300 5300 4700
+	5000 4650 5300 4650
+Wire Wire Line
+	5300 4650 5650 4650
+Wire Wire Line
+	5300 4300 5300 4650
+Wire Wire Line
+	5300 4650 5300 4700
 Wire Wire Line
 	5650 4650 5650 4700
@@
 Connection ~ 6900 4750
 Wire Wire Line
-	3800 5900 8400 5900
+	3800 5900 6900 5900
+Wire Wire Line
+	6900 5900 8400 5900
 Wire Wire Line
 	3800 5900 3800 5600
@@
 	8200 5550 8400 5550
 Wire Wire Line
-	6900 4950 6900 7050
+	6900 4950 6900 5900
+Wire Wire Line
+	6900 5900 6900 7050
 Connection ~ 6900 5900
 $Comp
@@
 $EndComp
 Wire Wire Line
+	8600 4200 8600 5450
+Wire Wire Line
 	8600 5450 8600 5950
 $Comp
@@
 P 9400 6300
 F 0 "D47" H 9400 6400 40  0000 C CNN
-F 1 "DIODE" H 9400 6200 40  0000 C CNN
+F 1 "DIODE" H 9400 6200 40  0001 C CNN
 F 2 "~" H 9400 6300 60  0000 C CNN
 F 3 "~" H 9400 6300 60  0000 C CNN
@@
 P 9600 6500
 F 0 "D48" H 9600 6600 40  0000 C CNN
-F 1 "DIODE" H 9600 6400 40  0000 C CNN
+F 1 "DIODE" H 9600 6400 40  0001 C CNN
 F 2 "~" H 9600 6500 60  0000 C CNN
 F 3 "~" H 9600 6500 60  0000 C CNN
@@
 P 10000 5200
 F 0 "D46" H 10000 5300 40  0000 C CNN
-F 1 "DIODE" H 10000 5100 40  0000 C CNN
+F 1 "DIODE" H 10000 5100 40  0001 C CNN
 F 2 "~" H 10000 5200 60  0000 C CNN
 F 3 "~" H 10000 5200 60  0000 C CNN
@@
 P 9800 5000
 F 0 "D45" H 9800 5100 40  0000 C CNN
-F 1 "DIODE" H 9800 4900 40  0000 C CNN
+F 1 "DIODE" H 9800 4900 40  0001 C CNN
 F 2 "~" H 9800 5000 60  0000 C CNN
 F 3 "~" H 9800 5000 60  0000 C CNN
@@
 Connection ~ 10000 5000
 Wire Wire Line
-	9600 5000 8550 5000
-Wire Wire Line
-	8550 5000 8550 4450
-Wire Wire Line
-	8550 4450 6550 4450
+	9600 5000 9600 5000
+Wire Wire Line
+	9600 5000 9600 4450
+Wire Wire Line
+	9600 4450 6550 4450
 $Comp
 L USR R45
@@
 $EndComp
 Wire Wire Line
-	10000 5000 10250 5000
+	10000 5000 10200 5000
+Wire Wire Line
+	10200 5000 10250 5000
 $Comp
 L +5V #PWR0173
@@
 $EndComp
 Connection ~ 10200 4500
-Wire Wire Line
-	9850 1200 9700 1200
 NoConn ~ 8400 1950
 NoConn ~ 8500 1950
 NoConn ~ 8600 1950
 NoConn ~ 8700 1950
-NoConn ~ 8800 1950
-NoConn ~ 8900 1950
-NoConn ~ 9000 1950
-NoConn ~ 9100 1950
 Text Notes 2800 1000 0    60   ~ 0
 DATA
@@
 Connection ~ 10000 3650
 Wire Wire Line
-	9700 700  9700 1850
-Wire Wire Line
-	9700 700  7800 700
+	7800 700  9750 700
+Wire Wire Line
+	9750 700  10400 700
 Wire Wire Line
 	7800 700  7800 1100
 Wire Wire Line
 	7800 1100 8000 1100
-Connection ~ 9700 1200
-Text Notes 11950 3100 1    60   ~ 0
-DETECT SECRET WORD
 Wire Wire Line
 	1350 4500 1350 4250
@@
 	7250 1250 7250 4200
 Wire Wire Line
-	7250 4200 8350 4200
-Wire Wire Line
-	8350 4200 8350 5450
-Connection ~ 8350 5450
-Wire Wire Line
-	9700 1850 10000 1850
+	7250 4200 8550 4200
+Wire Wire Line
+	8550 4200 8600 4200
 Wire Wire Line
 	10000 5000 10000 4550
 Wire Wire Line
 	10000 1850 10000 2750
+$Comp
+L 4585 U?
+U 1 1 5BFDEC59
+P 8600 2750
+F 0 "U?" H 8800 3350 60  0000 C CNN
+F 1 "4585" H 8750 2050 60  0000 C CNN
+F 2 "~" H 8750 2750 60  0000 C CNN
+F 3 "~" H 8750 2750 60  0000 C CNN
+	1    8600 2750
+	0    1    1    0
+$EndComp
+$Comp
+L USGND #PWR?
+U 1 1 5BFDEC66
+P 8450 2200
+F 0 "#PWR?" H 8450 2200 30  0001 C CNN
+F 1 "USGND" H 8450 2130 30  0001 C CNN
+F 2 "~" H 8450 2200 60  0000 C CNN
+F 3 "~" H 8450 2200 60  0000 C CNN
+	1    8450 2200
+	-1   0    0    1
+$EndComp
+Connection ~ 8450 2200
+$Comp
+L USGND #PWR?
+U 1 1 5BFDEC6C
+P 8650 2200
+F 0 "#PWR?" H 8650 2200 30  0001 C CNN
+F 1 "USGND" H 8650 2130 30  0001 C CNN
+F 2 "~" H 8650 2200 60  0000 C CNN
+F 3 "~" H 8650 2200 60  0000 C CNN
+	1    8650 2200
+	-1   0    0    1
+$EndComp
+Connection ~ 8650 2200
+Wire Wire Line
+	9100 1950 9100 2200
+Wire Wire Line
+	9000 1950 9000 2200
+Wire Wire Line
+	8900 1950 8900 2200
+Wire Wire Line
+	8800 1950 8800 2200
+$Comp
+L +5V #PWR?
+U 1 1 5BFDEDF2
+P 8000 2200
+F 0 "#PWR?" H 8000 2290 20  0001 C CNN
+F 1 "+5V" H 8000 2290 30  0000 C CNN
+F 2 "" H 8000 2200 60  0000 C CNN
+F 3 "" H 8000 2200 60  0000 C CNN
+	1    8000 2200
+	1    0    0    -1
+$EndComp
+$Comp
+L +5V #PWR?
+U 1 1 5BFDEDF8
+P 8100 2200
+F 0 "#PWR?" H 8100 2290 20  0001 C CNN
+F 1 "+5V" H 8100 2290 30  0000 C CNN
+F 2 "" H 8100 2200 60  0000 C CNN
+F 3 "" H 8100 2200 60  0000 C CNN
+	1    8100 2200
+	1    0    0    -1
+$EndComp
+$Comp
+L USGND #PWR?
+U 1 1 5BFDEDFE
+P 8200 2200
+F 0 "#PWR?" H 8200 2200 30  0001 C CNN
+F 1 "USGND" H 8200 2130 30  0001 C CNN
+F 2 "~" H 8200 2200 60  0000 C CNN
+F 3 "~" H 8200 2200 60  0000 C CNN
+	1    8200 2200
+	-1   0    0    1
+$EndComp
+$Comp
+L USGND #PWR?
+U 1 1 5BFDEE04
+P 8300 2200
+F 0 "#PWR?" H 8300 2200 30  0001 C CNN
+F 1 "USGND" H 8300 2130 30  0001 C CNN
+F 2 "~" H 8300 2200 60  0000 C CNN
+F 3 "~" H 8300 2200 60  0000 C CNN
+	1    8300 2200
+	-1   0    0    1
+$EndComp
+Connection ~ 8000 2200
+Connection ~ 8100 2200
+Connection ~ 8200 2200
+Connection ~ 8300 2200
+Text Notes 7800 3000 1    60   ~ 0
+DETECT SECRET WORD
+$Comp
+L USGND #PWR?
+U 1 1 5BFDF148
+P 8550 2200
+F 0 "#PWR?" H 8550 2200 30  0001 C CNN
+F 1 "USGND" H 8550 2130 30  0001 C CNN
+F 2 "~" H 8550 2200 60  0000 C CNN
+F 3 "~" H 8550 2200 60  0000 C CNN
+	1    8550 2200
+	-1   0    0    1
+$EndComp
+Connection ~ 8550 2200
+$Comp
+L DIODE D?
+U 1 1 5BFDF2F2
+P 8750 3550
+F 0 "D?" H 8750 3650 40  0000 C CNN
+F 1 "DIODE" H 8750 3450 40  0001 C CNN
+F 2 "~" H 8750 3550 60  0000 C CNN
+F 3 "~" H 8750 3550 60  0000 C CNN
+	1    8750 3550
+	-1   0    0    1
+$EndComp
+NoConn ~ 8450 3300
+NoConn ~ 8650 3300
+Wire Wire Line
+	8550 3300 8550 3550
+$Comp
+L DIODE D?
+U 1 1 5BFDF35D
+P 8750 3800
+F 0 "D?" H 8750 3900 40  0000 C CNN
+F 1 "DIODE" H 8750 3700 40  0001 C CNN
+F 2 "~" H 8750 3800 60  0000 C CNN
+F 3 "~" H 8750 3800 60  0000 C CNN
+	1    8750 3800
+	-1   0    0    1
+$EndComp
+Connection ~ 8600 5450
+Wire Wire Line
+	8550 3800 8550 4200
+Connection ~ 8550 4200
+Wire Wire Line
+	8950 3550 8950 3800
+$Comp
+L USR R?
+U 1 1 5BFDF4A3
+P 9200 3800
+F 0 "R?" V 9280 3800 40  0000 C CNN
+F 1 "100K" V 9100 3800 40  0000 C CNN
+F 2 "~" V 9130 3800 30  0000 C CNN
+F 3 "~" H 9200 3800 30  0000 C CNN
+	1    9200 3800
+	0    -1   -1   0
+$EndComp
+Connection ~ 8950 3800
+$Comp
+L +5V #PWR?
+U 1 1 5BFDF4AE
+P 9450 3800
+F 0 "#PWR?" H 9450 3890 20  0001 C CNN
+F 1 "+5V" H 9450 3890 30  0000 C CNN
+F 2 "" H 9450 3800 60  0000 C CNN
+F 3 "" H 9450 3800 60  0000 C CNN
+	1    9450 3800
+	0    1    1    0
+$EndComp
+Connection ~ 9450 3800
+Wire Wire Line
+	9850 1300 9750 1300
+Wire Wire Line
+	9750 1300 9750 3550
+Wire Wire Line
+	9750 3550 8950 3550
+Wire Wire Line
+	10400 700  10400 1850
+Wire Wire Line
+	10400 1850 10000 1850
+Wire Wire Line
+	9750 700  9750 1200
+Wire Wire Line
+	9750 1200 9850 1200
+Connection ~ 9750 700
 $EndSCHEMATC

Commit message: added rs232 output buffer
Parts:
- added Q?: MOSFET_N, ~, symbol MOSFET_N
- added Q?: MOSFET_P, ~, symbol MOSFET_P
- added R?: 100K, ~, symbol USR
Connections:
- wire segments 66 -> 63
Changed lines of the file:
@@
 Connection ~ 9500 1400
 Wire Wire Line
-	2650 4500 2700 4500
-Wire Wire Line
-	2700 4500 2750 4500
+	2650 4500 2750 4500
 Wire Wire Line
 	3250 4500 3800 4500
@@
 Connection ~ 5800 4300
 Wire Wire Line
-	5000 4650 5300 4650
-Wire Wire Line
-	5300 4650 5650 4650
-Wire Wire Line
-	5300 4300 5300 4650
-Wire Wire Line
-	5300 4650 5300 4700
+	5000 4650 5650 4650
+Wire Wire Line
+	5300 4300 5300 4700
 Wire Wire Line
 	5650 4650 5650 4700
@@
 Connection ~ 6900 4750
 Wire Wire Line
-	3800 5900 6900 5900
-Wire Wire Line
-	6900 5900 8400 5900
+	3800 5900 8400 5900
 Wire Wire Line
 	3800 5900 3800 5600
@@
 	8200 5550 8400 5550
 Wire Wire Line
-	6900 4950 6900 5900
-Wire Wire Line
-	6900 5900 6900 7050
+	6900 4950 6900 7050
 Connection ~ 6900 5900
 $Comp
@@
 $EndComp
 Wire Wire Line
-	8600 4200 8600 5450
-Wire Wire Line
-	8600 5450 8600 5950
+	8600 4200 8600 5950
 $Comp
 L USGND #PWR0170
@@
 $EndComp
 Wire Wire Line
-	10000 5000 10200 5000
-Wire Wire Line
-	10200 5000 10250 5000
+	10000 5000 10250 5000
 $Comp
 L +5V #PWR0173
@@
 Connection ~ 10000 3650
 Wire Wire Line
-	7800 700  9750 700
-Wire Wire Line
-	9750 700  10400 700
+	7800 700  10400 700
 Wire Wire Line
 	7800 700  7800 1100
@@
 	7250 1250 7250 4200
 Wire Wire Line
-	7250 4200 8550 4200
-Wire Wire Line
-	8550 4200 8600 4200
+	7250 4200 8600 4200
 Wire Wire Line
 	10000 5000 10000 4550
@@
 	9850 1300 9750 1300
 Wire Wire Line
-	9750 1300 9750 3550
-Wire Wire Line
-	9750 3550 8950 3550
-Wire Wire Line
 	10400 700  10400 1850
 Wire Wire Line
@@
 	9750 1200 9850 1200
 Connection ~ 9750 700
+$Comp
+L MOSFET_N Q?
+U 1 1 5BFE02AA
+P 9550 2900
+F 0 "Q?" H 9560 3070 60  0000 R CNN
+F 1 "MOSFET_N" H 9560 2750 60  0000 R CNN
+F 2 "~" H 9550 2900 60  0000 C CNN
+F 3 "~" H 9550 2900 60  0000 C CNN
+	1    9550 2900
+	0    -1   -1   0
+$EndComp
+Wire Wire Line
+	8950 3550 9550 3550
+Wire Wire Line
+	9550 3550 9550 3100
+$Comp
+L USGND #PWR?
+U 1 1 5BFE032C
+P 9750 2800
+F 0 "#PWR?" H 9750 2800 30  0001 C CNN
+F 1 "USGND" H 9750 2730 30  0001 C CNN
+F 2 "~" H 9750 2800 60  0000 C CNN
+F 3 "~" H 9750 2800 60  0000 C CNN
+	1    9750 2800
+	0    -1   -1   0
+$EndComp
+Connection ~ 9750 2800
+$Comp
+L MOSFET_P Q?
+U 1 1 5BFE0334
+P 9550 1850
+F 0 "Q?" H 9550 2040 60  0000 R CNN
+F 1 "MOSFET_P" H 9550 1670 60  0000 R CNN
+F 2 "~" H 9550 1850 60  0000 C CNN
+F 3 "~" H 9550 1850 60  0000 C CNN
+	1    9550 1850
+	0    -1   -1   0
+$EndComp
+Wire Wire Line
+	9350 2800 9350 2700
+Wire Wire Line
+	9350 2700 9550 2700
+Wire Wire Line
+	9550 2700 9550 2050
+$Comp
+L USR R?
+U 1 1 5BFE03C0
+P 9350 2450
+F 0 "R?" V 9430 2450 40  0000 C CNN
+F 1 "100K" V 9250 2450 40  0000 C CNN
+F 2 "~" V 9280 2450 30  0000 C CNN
+F 3 "~" H 9350 2450 30  0000 C CNN
+	1    9350 2450
+	-1   0    0    1
+$EndComp
+Connection ~ 9350 2700
+$Comp
+L +5V #PWR?
+U 1 1 5BFE03C6
+P 9350 2200
+F 0 "#PWR?" H 9350 2290 20  0001 C CNN
+F 1 "+5V" H 9350 2290 30  0000 C CNN
+F 2 "" H 9350 2200 60  0000 C CNN
+F 3 "" H 9350 2200 60  0000 C CNN
+	1    9350 2200
+	1    0    0    -1
+$EndComp
+Connection ~ 9350 2200
+Wire Wire Line
+	9350 1750 9350 1550
+Wire Wire Line
+	9350 1550 9750 1550
+Wire Wire Line
+	9750 1550 9750 1300
+$Comp
+L +5V #PWR?
+U 1 1 5BFE044A
+P 9750 1750
+F 0 "#PWR?" H 9750 1840 20  0001 C CNN
+F 1 "+5V" H 9750 1840 30  0000 C CNN
+F 2 "" H 9750 1750 60  0000 C CNN
+F 3 "" H 9750 1750 60  0000 C CNN
+	1    9750 1750
+	0    1    1    0
+$EndComp
+Connection ~ 9750 1750
 $EndSCHEMATC

Commit message: simplified RS232, bench test successful, needs tested against actual logic board
Parts:
- removed D? (x2): DIODE, ~, symbol DIODE
- removed Q?: MOSFET_N, ~, symbol MOSFET_N
- removed Q?: MOSFET_P, ~, symbol MOSFET_P
- removed R? (x2): 100K, ~, symbol USR
Connections:
- wire segments 63 -> 66
