File: schematic/rs232-board.sch (KiCad schematic (older format))
At the start: 21 parts, among them Q7 MOSFET_P, U28 4094, U29 4017, U89 4013, U99 4584

Commit message: RS232 board REV 3
Parts:
- removed R43: 1K3 1%, ~, symbol USR
- added C?: 1uF, ~, symbol C
- added C?: 20pF, ~, symbol CSMALL
- added D?: LED, ~, symbol LED
- added D?: DIODE, ~, symbol DIODE
- added R?: 1K, ~, symbol USR
- added U?: AZ2940T-3.3E1, symbol LM7805
- C?: value 10pF -> 20pF
- R42: value 47K 1% -> 97K6 1%
- R45: value 10K -> 100K
- RV1: value 470R -> 5K
Connections:
- wire segments 66 -> 58
Other:
- note added: "3.3V"
- note added: "AS BUILT VALUE: 101K1"
- note added: "EXACT RESISTANCE DETERMINED AT ASSEMBLY"
- note removed: "TARGET VALUE APPROX. 48K7"
