File: schematic/logic-clock.kicad_pcb (KiCad board)
At the start: 2 copper layers, 0 parts

Commit message: started pcb
Parts:
- added AFF1: 7SEG-KB, 7SEG-KB, F.Cu at (227.3, 44.5)
- added P5: 4-PIN_HEADER, PIN_ARRAY_4x1, F.Cu at (222.2, 74.9)
- added P6: 2-PIN_HEADER, PIN_ARRAY_2X1, F.Cu at (241.3, 66.0)
- added U6: 4511, DIP-16__300_ELL, F.Cu at (227.3, 66.0)
Routing:
- net GND: track 0.00 -> 114.7 mm
- net N-0000079: track 0.00 -> 71.0 mm
- net N-0000072: track 0.00 -> 32.5 mm
- net +5V: track 0.00 -> 32.3 mm
- net N-0000076: track 0.00 -> 31.0 mm
- net N-0000073: track 0.00 -> 30.3 mm
- net N-0000075: track 0.00 -> 28.8 mm
- net (no net): track 25.3 -> 0.00 mm
- net /display-board/0A: track 0.00 -> 20.2 mm
- net N-0000077: track 0.00 -> 20.1 mm
- net N-0000078: track 0.00 -> 10.7 mm
- net /display-board/0D: track 0.00 -> 7.93 mm
- net /display-board/0C: track 0.00 -> 6.13 mm
- net /display-board/0B: track 0.00 -> 6.13 mm
Other:
- net class Default: trace_width 0.254 -> 0.762
- net class tiny added: clearance 0.254, trace_width 0.254, via_dia 0.889, via_drill 0.635

Commit message: pcb rev 1
Parts:
- added AFF2: AM-PM, 7SEG-KB, F.Cu at (47.0, 90.2)
- added AFF3: TEN-HOURS, 7SEG-KB, F.Cu at (77.5, 90.2)
- added AFF4: HOURS, 7SEG-KB, F.Cu at (105.4, 90.2)
- added AFF5: TEN-MINUTES, 7SEG-KB, F.Cu at (135.9, 90.2)
- added AFF6: MINUTES, 7SEG-KB, F.Cu at (163.8, 90.2)
- added AFF7: TEN-SECONDS, 7SEG-KB, F.Cu at (194.3, 90.2)
- added AFF8: SECONDS, 7SEG-KB, F.Cu at (222.2, 90.2)
- added C12: 100nF BYPASS, C1, F.Cu at (121.9, 111.8)
- added C13: 100nF BYPASS, C1, F.Cu at (149.9, 111.8)
- added C14: 100nF BYPASS, C1, F.Cu at (180.3, 111.8)
- added C15: 100nF BYPASS, C1, F.Cu at (208.3, 111.8)
- added C16: 100nF BYPASS, C1, F.Cu at (236.2, 111.8)
- added C17: 100nF BYPASS, C1, F.Cu at (91.4, 111.8)
- added D24: LED, LED-5MM, F.Cu at (120.7, 83.8)
- added D25: LED, LED-5MM, F.Cu at (120.7, 96.5)
- added D26: LED, LED-5MM, F.Cu at (179.1, 83.8)
- added D27: LED, LED-5MM, F.Cu at (179.1, 96.5)
- added P13: 2-PIN_HEADER, PIN_ARRAY_2X1, F.Cu at (69.8, 120.7)
- added P14: 4-PIN_HEADER, PIN_ARRAY_4x1, F.Cu at (100.3, 120.7)
- added P15: 4-PIN_HEADER, PIN_ARRAY_4x1, F.Cu at (130.8, 120.7)
- added P16: 4-PIN_HEADER, PIN_ARRAY_4x1, F.Cu at (158.8, 120.7)
- added P17: 4-PIN_HEADER, PIN_ARRAY_4x1, F.Cu at (189.2, 120.7)
- added P18: 4-PIN_HEADER, PIN_ARRAY_4x1, F.Cu at (217.2, 120.7)
- added Q2: MOS_P, TO92DGS, F.Cu at (62.2, 91.4)
- added Q3: ZVN4206, TO92DGS, F.Cu at (78.7, 119.4)
- added R27: 1K, R3-LARGE_PADS, F.Cu at (59.7, 105.4)
- added R28: 1K, R3-LARGE_PADS, F.Cu at (77.5, 110.5)
- added R29: 1K, R1, F.Cu at (120.7, 90.2)
- added R30: 1K, R1, F.Cu at (179.1, 90.2)
- added R31: 1K, R3-LARGE_PADS, F.Cu at (234.9, 91.4)
- added U10: 4511, DIP-16__300_ELL, F.Cu at (135.9, 111.8)
- added U11: 4511, DIP-16__300_ELL, F.Cu at (163.8, 111.8)
- added U12: 4511, DIP-16__300_ELL, F.Cu at (194.3, 111.8)
- added U13: 4511, DIP-16__300_ELL, F.Cu at (222.2, 111.8)
- added U9: 4511, DIP-16__300_ELL, F.Cu at (105.4, 111.8)
- AFF1: value 7SEG-KB -> TENTH-SECONDS
- moved P6 57.4 mm to (259.1, 120.7), turned to 0 degrees
- moved P5 51.1 mm to (245.1, 120.7)
- moved AFF1 51.1 mm to (250.2, 90.2)
- moved U6 51.1 mm to (250.2, 111.8)
Routing:
- net GND: track 114.7 -> 893.0 mm
- net +5V: track 32.3 -> 644.5 mm
- net N-00000138: track 0.00 -> 49.4 mm
- net N-00000141: track 0.00 -> 47.9 mm
- net N-0000099: track 0.00 -> 34.8 mm
- net N-00000173: track 0.00 -> 34.8 mm
- net N-00000162: track 0.00 -> 34.8 mm
- net N-00000107: track 0.00 -> 34.8 mm
- net N-00000118: track 0.00 -> 31.3 mm
- net N-0000094: track 0.00 -> 31.3 mm
- net N-00000169: track 0.00 -> 31.3 mm
- net N-00000157: track 0.00 -> 31.3 mm
- net N-00000112: track 0.00 -> 31.3 mm
- net N-00000124: track 0.00 -> 30.6 mm
- net /display-board/AM: track 0.00 -> 30.0 mm
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Other:
- net class tiny removed

Commit message: pcb rev 2
Routing:
- net N-00000150: track 71.0 -> 31.3 mm
- net N-00000155: track 30.3 -> 26.2 mm
- net N-00000153: track 34.4 -> 30.6 mm
- net N-00000145: track 28.8 -> 25.2 mm
- net N-00000152: track 20.1 -> 17.6 mm
- net N-00000146: track 31.0 -> 28.8 mm
- net GND: track 893.0 -> 892.0 mm
- net /display-board/0A: track 20.2 -> 20.9 mm
Other:
- net class Default: trace_width 0.762 -> 0.254

Commit message: pcb rev 3
Parts:
- R31: footprint R3-LARGE_PADS -> R1
- moved Q2 24.4 mm to (73.7, 113.0)
- moved AFF2 19.1 mm to (66.0, 90.2)
- moved AFF3 16.5 mm to (94.0, 90.2)
- moved P13 16.5 mm to (86.4, 120.7)
- moved Q3 16.5 mm to (95.2, 119.4)
- moved R28 16.5 mm to (94.0, 110.5)
- moved AFF4 12.7 mm to (118.1, 90.2)
- moved C17 12.7 mm to (104.1, 111.8)
- moved P14 12.7 mm to (113.0, 120.7)
- moved U9 12.7 mm to (118.1, 111.8)
- moved D24 11.4 mm to (132.1, 83.8)
- moved D25 11.4 mm to (132.1, 96.5)
- moved R29 11.4 mm to (132.1, 90.2)
- moved C12 10.9 mm to (128.3, 120.7), turned to 180 degrees
- moved C13 10.2 mm to (154.9, 120.7), turned to 180 degrees
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Routing:
- net GND: track 892.0 -> 796.7 mm
- net +5V: track 644.7 -> 662.3 mm
- net N-00000117: track 6.35 -> 23.9 mm
- net /display-board/AM: track 30.0 -> 12.8 mm
- net /display-board/0C: track 6.13 -> 9.94 mm
- net /display-board/0B: track 6.13 -> 9.94 mm
- net /display-board/0D: track 7.93 -> 5.61 mm
- net N-00000141: track 47.9 -> 49.9 mm
- net /display-board/0A: track 20.9 -> 19.0 mm
- net /display-board/1D: track 7.93 -> 8.67 mm
- net N-00000176: track 5.08 -> 4.44 mm

Commit message: lots of stuff
Parts:
- U10, U11, U12, U13, U6, U9: footprint DIP-16__300_ELL -> DIP-16__300
Other:
- net class Default: clearance 0.254 -> 0.381
- rule trace_clearance: 0.254 -> 0.381

Commit message: ready to lay out pcb
Parts:
- removed AFF1: TENTH-SECONDS, 7SEG-KB
- removed AFF2: AM-PM, 7SEG-KB
- removed AFF3: TEN-HOURS, 7SEG-KB
- removed AFF4: HOURS, 7SEG-KB
- removed AFF5: TEN-MINUTES, 7SEG-KB
- removed AFF6: MINUTES, 7SEG-KB
- removed AFF7: TEN-SECONDS, 7SEG-KB
- removed AFF8: SECONDS, 7SEG-KB
- removed C12, C13, C14, C15: 100nF BYPASS, C1
- removed P5: 4-PIN_HEADER, PIN_ARRAY_4x1
- removed P6: 2-PIN_HEADER, PIN_ARRAY_2X1
- removed Q2: MOS_P, TO92DGS
- removed R27, R28: 1K, R3-LARGE_PADS
- removed U10, U11, U12, U6, U9: 4511, DIP-16__300
- added C18: 100nF, C1, F.Cu at (-34.0, -38.6)
- added C19: 100nF, C1, F.Cu at (18.8, -35.1)
- added C20: 100nF, C1, F.Cu at (34.0, -41.1)
- added C21: 100nF, C1, F.Cu at (2.03, -22.9)
- added C22: 100nF, C1, F.Cu at (53.8, -33.0)
- added C23: 100nF, C1, F.Cu at (-10.2, -33.0)
- added C24: 100nF, C1, F.Cu at (-94.5, -13.7)
- added C25: 100nF, C1, F.Cu at (-90.9, -47.2)
- added C26: 100nF, C1, F.Cu at (-70.6, -54.9)
- added C27: 100nF, C1, F.Cu at (-107.2, -13.7)
- added C28: 100nF, C1, F.Cu at (70.6, -43.2)
- added C29: 100nF, C1, F.Cu at (-49.8, 15.7)
- added C30: 100nF, C1, F.Cu at (-13.2, -12.7)
- added D28: DIODE, D3, F.Cu at (-67.6, 13.2)
- added D29: DIODE, D3, F.Cu at (61.5, -22.4)
- added D30: DIODE, D3, F.Cu at (81.3, -32.5)
- added D31: DIODE, D3, F.Cu at (67.6, 17.8)
- added D32: DIODE, D3, F.Cu at (51.3, 18.3)
- added D33: DIODE, D3, F.Cu at (104.6, 3.56)
- added D34: DIODE, D3, F.Cu at (10.2, -11.7)
- added D35: DIODE, D3, F.Cu at (76.2, -12.2)
- added D36: DIODE, D3, F.Cu at (-10.7, 50.3)
- added D37: DIODE, D3, F.Cu at (118.4, 17.3)
- added P11: 3-PIN_HEADER, PIN_ARRAY_3X1, F.Cu at (-14.2, 35.1)
- added P12: 2-PIN_HEADER, PIN_ARRAY_2X1, F.Cu at (-65.5, 30.0)
- added P19: 4-PIN_HEADER, PIN_ARRAY_4x1, F.Cu at (-34.5, -2.54)
- added P20: 3-PIN_HEADER, PIN_ARRAY_3X1, F.Cu at (104.6, -11.2)
- added P21: 4-PIN_HEADER, PIN_ARRAY_4x1, F.Cu at (43.2, -12.2)
- added P22: 3-PIN_HEADER, PIN_ARRAY_3X1, F.Cu at (-28.4, 27.4)
- added Q5: ZVN4206, TO92DGS, F.Cu at (41.1, 39.6)
- added Q6: ZVN4206, TO92DGS, F.Cu at (23.9, 29.0)
- added R32: 100K, R1, F.Cu at (57.4, 2.54)
- added R33: 100K, R1, F.Cu at (72.6, 4.06)
- added R34: 100K, R1, F.Cu at (194.6, 21.8)
- added R35: 100K, R1, F.Cu at (128.5, 26.9)
- added R36: 100K, R1, F.Cu at (82.8, 4.57)
- added RR1: 100K, SIL-9, F.Cu at (54.9, 27.4)
- added RR2: 100K, SIL-9, F.Cu at (87.9, 26.9)
- added U14: 4094, DIP-16__300, F.Cu at (224.5, 87.9)
- added U15: 4071, DIP-14__300, F.Cu at (125.5, 113.8)
- added U16: 4013, DIP-14__300, F.Cu at (90.4, 136.1)
- added U17: 4081, DIP-14__300, F.Cu at (32.0, 88.9)
- added U18: 4029, DIP-16__300, F.Cu at (113.3, 46.7)
- added U19: 4029, DIP-16__300, F.Cu at (174.8, 74.7)
- added U20: 4029, DIP-16__300, F.Cu at (156.5, 26.4)
- added U21: 4029, DIP-16__300, F.Cu at (84.3, 86.9)
- added U22: 4518, DIP-16__300, F.Cu at (171.7, 115.3)
- added U23: 4071, DIP-14__300, F.Cu at (208.3, 145.3)
- added U24: 4584, DIP-14__300, F.Cu at (146.3, 159.5)
- added U25: 4072, DIP-14__300, F.Cu at (42.7, 141.2)
- C16: value 100nF BYPASS -> 1uF
- C17: value 100nF BYPASS -> 100nF
- D24, D26, D27: value LED -> DIODE; footprint LED-5MM -> D3
- P13: value 2-PIN_HEADER -> 3-PIN_HEADER; footprint PIN_ARRAY_2X1 -> PIN_ARRAY_3X1
- P14: value 4-PIN_HEADER -> 1-PIN_HEADER; footprint PIN_ARRAY_4x1 -> PIN_ARRAY_1
- R30, R31: value 1K -> 100K
- U13: value 4511 -> 4094
- moved C16 341.1 mm to (-77.7, -25.4), turned to 0 degrees
- moved P18 270.7 mm to (-33.0, 17.3)
- moved P16 244.0 mm to (-41.1, -9.65)
- moved P14 219.7 mm to (-66.0, -6.60)
- moved P17 219.2 mm to (24.4, -19.3)
- moved D27 209.0 mm to (-9.65, 18.3), turned to 0 degrees
- moved C17 208.2 mm to (-49.8, -28.4), turned to 0 degrees
- moved P15 205.1 mm to (-31.5, 9.65)
- moved D24 184.7 mm to (-2.03, -43.2), turned to 0 degrees
- moved D26 163.1 mm to (35.1, 17.8), turned to 0 degrees
- moved P13 147.0 mm to (-38.6, 43.2)
- moved D25 145.8 mm to (256.0, 19.8), turned to 0 degrees
- moved R31 135.4 mm to (117.9, 27.4), turned to 0 degrees
- moved Q3 94.7 mm to (25.4, 55.4), turned to 0 degrees
- moved R30 75.5 mm to (133.1, 34.5), turned to 0 degrees
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Connections:
- D24 pad 1: N-00000102 -> GND
- D24 pad 2: GND -> +5V
- D25 pad 1: N-00000102 -> N-00000225
- D26 pad 1: N-00000175 -> /display-board/1A
- D26 pad 2: GND -> N-00000224
- D27 pad 1: N-00000175 -> /display-board/0A
- D27 pad 2: GND -> N-00000222
- P13 pad 1: /display-board/AM -> 1Hz
- P13 pad 2: /display-board/TEN-HR -> /logic-board/SEC_CLOCK
- P14 pad 1: /display-board/5A -> 1Hz
- P15 pad 1: /display-board/4A -> /comparator-board/4A
- P15 pad 2: /display-board/4B -> /comparator-board/4B
- P15 pad 3: /display-board/4C -> /comparator-board/4C
- P15 pad 4: /display-board/4D -> /comparator-board/4D
- P16 pad 1: /display-board/3A -> /comparator-board/3A
- P16 pad 2: /display-board/3B -> /comparator-board/3B
- P16 pad 3: /display-board/3C -> /comparator-board/3C
- P16 pad 4: /display-board/3D -> /comparator-board/3D
- Q3 pad G: /display-board/TEN-HR -> /comparator-board/TEN-HOURS
- Q3 pad S: GND -> DPS
- R29 pad 1: +5V -> N-00000225
- R29 pad 2: N-00000102 -> +5V
- R30 pad 1: +5V -> GND
- R30 pad 2: N-00000175 -> SET
- R31 pad 1: +5V -> N-00000223
- R31 pad 2: N-00000176 -> +5V
- U13 pad 1: /display-board/1B -> SET
- U13 pad 10: N-00000122 -> (no net)
- U13 pad 15: N-00000123 -> SET
- U13 pad 2: /display-board/1C -> /logic-board/DATA
- U13 pad 3: +5V -> /logic-board/CLOCK
- U13 pad 4: +5V -> N-00000200
- U13 pad 5: GND -> N-00000203
- U13 pad 6: /display-board/1D -> N-00000202
- U13 pad 7: /display-board/1A -> N-00000201
Routing:
- net GND: track 796.7 -> 0.00 mm
- net +5V: track 662.3 -> 0.00 mm
- net N-00000141: track 49.9 -> 0.00 mm
- net N-00000138: track 49.4 -> 0.00 mm
- net N-00000162: track 34.8 -> 0.00 mm
- net N-0000099: track 34.8 -> 0.00 mm
- net N-00000173: track 34.8 -> 0.00 mm
- net N-00000107: track 34.8 -> 0.00 mm
- net N-00000150: track 31.3 -> 0.00 mm
- net N-0000094: track 31.3 -> 0.00 mm
- net N-00000196: track 31.3 -> 0.00 mm
- net N-00000157: track 31.3 -> 0.00 mm
- net N-00000169: track 31.3 -> 0.00 mm
- net N-00000112 (its old number): track 31.3 -> 0.00 mm
- net N-00000195: track 30.6 -> 0.00 mm
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Other:
- net class Default: clearance 0.381 -> 0.254
- rule trace_clearance: 0.381 -> 0.254

Commit message: layout almost ready for routing
Parts:
- removed C30: 100nF, C1
- removed Q3: ZVN4206, TO92DGS
- moved C16 354.3 mm to (247.9, 114.3), turned to 90 degrees
- moved P14 346.2 mm to (254.0, 125.5)
- moved D28 329.8 mm to (231.6, 151.9)
- moved P13 307.0 mm to (254.0, 136.1), turned to 90 degrees
- moved P19 302.0 mm to (218.9, 161.5)
- moved P22 295.1 mm to (254.0, 112.8), turned to 90 degrees
- moved C27 293.5 mm to (138.2, 147.3), turned to 270 degrees
- moved D24 289.8 mm to (242.8, 111.8), turned to 270 degrees
- moved P18 278.5 mm to (205.2, 161.5)
- moved C25 261.2 mm to (107.7, 122.4), turned to 270 degrees
- moved D36 260.5 mm to (231.6, 145.8)
- moved P16 259.5 mm to (153.9, 161.5)
- moved C24 258.5 mm to (107.7, 147.3), turned to 270 degrees
- moved D27 254.4 mm to (217.4, 133.1)
- moved P17 240.5 mm to (182.9, 161.5)
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
Commit message: fixed unused chip connections
Connections:
- U16 pad 3: N-00000213 -> N-00000223
- U17 pad 12: (no net) -> GND
- U17 pad 13: (no net) -> GND
- U17 pad 5: (no net) -> GND
- U17 pad 6: (no net) -> GND
- U17 pad 8: (no net) -> GND
- U17 pad 9: (no net) -> GND
- U23 pad 12: (no net) -> GND
- U23 pad 13: (no net) -> GND
- U23 pad 8: (no net) -> GND
- U23 pad 9: (no net) -> GND
- U24 pad 10: N-00000245 -> (no net)
- U24 pad 11: N-00000256 -> GND
- U24 pad 13: (no net) -> GND
- U24 pad 3: /rs232-board/RS232-5V -> /comparator-board/5D
- U24 pad 4: N-00000247 -> N-00000223
- U24 pad 5: N-00000254 -> GND
- U24 pad 6: N-00000257 -> (no net)
- U24 pad 8: N-00000267 -> (no net)
- U24 pad 9: N-00000257 -> GND
